File: _autosave-STM32F429ZIT6.kicad_pcb (KiCad board)
At the start: 4 copper layers, 114.5 x 68.5 mm, 120 parts, among them J2 Conn_01x05_Pin, P1 Header 32X2, P2 Header 32X2, SW1 K3-1235S, U2 LD3985M33R, U3 MCP6004, U4 NAU88C22YG_C914209, U5 RCLAMP0521P.TCT_C3029033, U6 RCLAMP0521P.TCT_C3029033, U7 W9825G6KH-6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

Commit message: 18 errors left
Parts:
- moved C22 0.35 mm to (147.3, 84.0)
- moved R27 0.30 mm to (156.2, 77.3)
- moved D5 0.20 mm to (157.7, 77.0)
Routing:
- net /I2S_DOUT: track 95.7 -> 87.0 mm
- net +3.3V: track 78.6 -> 83.0 mm, vias 33 -> 35
- net Net-(U4-RHP): track 38.2 -> 41.1 mm
- net GND: track 82.7 -> 85.5 mm, vias 39 -> 47
- net Net-(U4-LHP): track 32.8 -> 35.2 mm
- removed copper zone on In2.Cu, net VDDA
