File: STM32F429ZIT6.kicad_sch (KiCad schematic)
At the start: 115 parts, among them J1 Conn_02x24_Odd_Even, J2 Conn_01x05_Pin, J3 Conn_02x16_Odd_Even, SW1 K3-1235S, U2 LD3985M33R, U3 MCP6004, U4 NAU88C22YG_C914209, U5 RCLAMP0521P.TCT_C3029033, U6 RCLAMP0521P.TCT_C3029033, U7 W9825G6KH-6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

Commit message: quick save
Parts:
- removed J1: Conn_02x24_Odd_Even, Connector_PinHeader_2.54mm:PinHeader_2x24_P2.54mm_Vertical, symbol Connector_Generic:Conn_02x24_Odd_Even
- removed J3: Conn_02x16_Odd_Even, Connector_PinHeader_2.54mm:PinHeader_2x16_P2.54mm_Vertical, symbol Connector_Generic:Conn_02x16_Odd_Even
- added J1, J3: Conn_02x30_Odd_Even, Connector_PinHeader_2.54mm:PinHeader_2x30_P2.54mm_Vertical, symbol Connector_Generic:Conn_02x30_Odd_Even
Connections:
- net PA0: now also J1.56 (Pin_56)
- net PA1: now also J1.58 (Pin_58)
- net PA10: now also J3.15 (Pin_15)
- net PA11: now also J3.13 (Pin_13)
- net PA12: now also J3.11 (Pin_11)
- net PA2: now also J1.60 (Pin_60)
- net PA3: now also J3.59 (Pin_59)
- net PA4: now also J3.57 (Pin_57)
- net PA5: now also J3.55 (Pin_55)
- net PA6: now also J3.53 (Pin_53)
- net PA7: now also J3.51 (Pin_51)
- net PA9: now also J3.17 (Pin_17)
- net PB0: now also J3.45 (Pin_45)
- net PB1: now also J3.43 (Pin_43)
- net PB10: now also J3.39 (Pin_39)
- net PB11: now also J3.37 (Pin_37)
- net PB12: now also J3.35 (Pin_35)
- net PB13: now also J3.33 (Pin_33)
- net PB2: now also J3.41 (Pin_41)
- net PB4: now also J1.16 (Pin_16)
- net PB7: now also J1.18 (Pin_18)
- net PB8: now also J1.20 (Pin_20)
- net PB9: now also J1.22 (Pin_22)
- net PC1: now also J1.50 (Pin_50)
- net PC13: now also J1.34 (Pin_34)
- net PC14: now also J1.36 (Pin_36)
- net PC15: now also J1.38 (Pin_38)
- net PC2: now also J1.52 (Pin_52)
- net PC3: now also J1.54 (Pin_54)
- net PC4: now also J3.49 (Pin_49)
- net PC5: now also J3.47 (Pin_47)
- net PC6: now also J3.21 (Pin_21)
- net PC8: now also J3.19 (Pin_19)
- net PD11: now also J3.31 (Pin_31)
- net PD12: now also J3.29 (Pin_29)
- net PD13: now also J3.27 (Pin_27)
- net PD2: now also J3.9 (Pin_9)
- net PD3: now also J3.7 (Pin_7)
- net PD4: now also J3.5 (Pin_5)
- net PD5: now also J3.3 (Pin_3)
- net PD6: now also J1.4 (Pin_4)
- net PD7: now also J1.6 (Pin_6)
- net PE2: now also J1.24 (Pin_24)
- net PE3: now also J1.26 (Pin_26)
- net PE4: now also J1.28 (Pin_28)
- net PE5: now also J1.30 (Pin_30)
- net PE6: now also J1.32 (Pin_32)
- net PF10: now also J1.48 (Pin_48)
- net PF6: now also J1.40 (Pin_40)
- net PF7: now also J1.42 (Pin_42)
- net PF8: now also J1.44 (Pin_44)
- net PF9: now also J1.46 (Pin_46)
- net PG10: now also J1.10 (Pin_10)
- net PG11: now also J1.12 (Pin_12)
- net PG12: now also J1.14 (Pin_14)
- net PG6: now also J3.25 (Pin_25)
- net PG7: now also J3.23 (Pin_23)
- net PG9: now also J1.8 (Pin_8)
Other:
- note added: "Conn_02x30_Odd_Even Connector_PinHeader_2.54mm:PinHeader_2x30_P2.54mm_Vertical"
- note removed: "Conn_02x16_Odd_Even Connector_PinHeader_2.54mm:PinHeader_2x16_P2.54mm_Vertical"

Commit message: KILL ME!!!!!!!!!!!
Parts:
- removed J1, J3: Conn_02x30_Odd_Even, Connector_PinHeader_2.54mm:PinHeader_2x30_P2.54mm_Vertical, symbol Connector_Generic:Conn_02x30_Odd_Even
- added P1, P2: Header 32X2, Connector_PinHeader_2.54mm:PinHeader_2x32_P2.54mm_Vertical, symbol MCD_TOOLS:root_0_Header 32X2_MCD_TOOLS.SchLib
- added SB26, SB27: Circuit Breaker, Jumper:SolderJumper-2_P1.3mm_Open_TrianglePad1.0x1.5mm, symbol MCD_TOOLS:root_0_Circuit Breaker_MCD_TOOLS.SCHLIB
Connections:
- net +3.3V: now also P1.22
- net A0: now also P1.7
- net A1: now also P1.8
- net A10: now also P2.35
- net A11: now also P2.38
- net A12: now also P2.62
- net A2: now also P1.5
- net A3: now also P1.6
- net A4: now also P1.3
- net A5: now also P1.4
- net A6: now also P2.31
- net A7: now also P2.34
- net A8: now also P2.33
- net A9: now also P2.36
- net BA0: now also P1.62
- net BA1: now also P1.61
- net BOOT0: now also P1.21
- net D0: now also P2.60
- net D1: now also P2.59
- net D10: now also P2.43
- net D11: now also P2.46
- net D12: now also P2.45
- net D13: now also P2.54
- net D14: now also P2.53
- net D15: now also P2.56
- net D2: now also P1.42
- net D3: now also P1.41
- net D4: now also P2.37
- net D5: now also P2.40
- net D6: now also P2.39
- net D7: now also P2.42
- net D8: now also P2.41
- net D9: now also P2.44
- net GND: now also P1.63, P1.64, P2.11, P2.29, P2.63, P2.64
- net I2S_BCLK: now also P1.45
- net I2S_DIN: now also P1.44
- net I2S_DOUT: now also P1.43
- net I2S_LRKCLK: now also P1.46
- net I2S_MCK: now also P1.56
- net I2S_SCL: now also P1.53
- net I2S_SDA: now also P1.54
- net LED_GREEN: now also P1.29
- net LED_RED: now also P1.30
- net NBL0: now also P1.17
- net NBL1: now also P1.18
- net NRST: now also P2.12
- net PA0: now also P2.18
- net PA1: now also P2.17
- net PA10: now also P1.51
- net PA11: now also P1.50
- net PA12: now also P1.49
- net PA2: now also P2.20
- net PA3: now also P2.19
- net PA4: now also P2.22
- net PA5: now also P2.21
- net PA6: now also P2.24
- net PA7: now also P2.23
- net PA9: now also P1.52
- net PB0: now also P2.28
- net PB1: now also P2.27
- net PB10: now also P2.48
- net PB11: now also P2.47
- net PB12: now also P2.50
- net PB13: now also P2.49
- net PB14: now also SB27.2
- net PB15: now also SB26.1
- net PB2: now also P2.30
- net PB4: now also P1.25
- net PB5: now also P1.26
- net PB6: now also P1.23
- net PB7: now also P1.24
- net PB8: now also P1.19
- net PB9: now also P1.20
- net PC0: now also P2.14
- net PC1: now also P2.13
- net PC13: now also P1.12
- net PC14: now also P1.9
- net PC15: now also P1.10
- net PC2: now also P2.16
- net PC3: now also P2.15
- net PC4: now also P2.26
- net PC5: now also P2.25
- net PC6: now also P1.57
- net PC8: now also P1.55
- net PD11: now also P2.55
- net PD12: now also P2.58
- net PD13: now also P2.57
- net PD2: now also P1.40
- net PD3: now also P1.39
- net PD4: now also P1.38
- net PD5: now also P1.37
- net PD6: now also P1.36
- net PD7: now also P1.35
- net PE2: now also P1.15
- net PE3: now also P1.16
- net PE4: now also P1.13
- net PE5: now also P1.14
- net PE6: now also P1.11
- net PF10: now also P2.7
- net PF11: now also P2.32
- net PF6: now also P2.3
- net PF7: now also P2.6
- net PF8: now also P2.5
- net PF9: now also P2.8
- net PG10: now also P1.34
- net PG11: now also P1.31
- net PG12: now also P1.32
- net PG15: now also P1.27
- net PG3: now also P2.61
- net PG6: now also P1.60
- net PG7: now also P1.59
- net PG8: now also P1.58
- net PG9: now also P1.33
- new net: P2.51, SB26.2
- new net: P2.52, SB27.1
- new net 3V: P2.1, P2.2
- new net 5V: P1.1, P1.2
- new net PA13: P1.48
- new net PA14: P1.47
- new net PB3: P1.28
- new net PH0: P2.10
- new net PH1: P2.9
- no-connect marks 3 -> 4
Other:
- note added: "3V"
- note added: "5V"
- note added: "BOOT1 / PB2"
- note added: "NC"

Commit message: getting closer, one side of the breakout is done ish for the sdram. still needs connections between the sdram and st chip
Parts:
- removed C26, C28: 100nF, PCM_JLCPCB:C_0402, symbol PCM_JLCPCB-Capacitors:0402,100nF
- added C26, C28: 1uF, PCM_JLCPCB:C_1206, symbol PCM_JLCPCB-Capacitors:1206,1uF
Connections:
- net GND: now also C26.2, C28.1
- net at C27.1, L1.2, R3.1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: now also C26.1
- net at C29.2, R3.2, U.1.32 (VREF+): now also C28.2
Other:
- note added: "extra pin!"
- moved on the sheet: D4, LED1, R27, R29

Commit message: closer to breakout done, need to wire codec now
Connections:
- net SWCLK is gone; now on net PA14: J2.3 (Pin_3), U.1.109 (PA14(JTCK-SWCLK))
- net SWDIO is gone; now on net PA13: J2.2 (Pin_2), U.1.105 (PA13(JTMS-SWDIO))
- net SWO is gone; now on net PB3: J2.4 (Pin_4), U.1.133 (PB3(JTDOTRACESWO))
Changed lines of the file:
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@@
 		)
 	)
+	(label "PA14"
+		(at 335.28 91.44 0)
+		(effects
+			(font
+				(size 1.27 1.27)
+			)
+			(justify left bottom)
+		)
+	)
 	(label "SDNWE"
 		(at 326.39 99.06 180)
@@
 		)
 	)
+	(label "PA13"
+		(at 335.28 88.9 0)
+		(effects
+			(font
+				(size 1.27 1.27)
+			)
+			(justify left bottom)
+		)
+	)
 	(label "PD10"
 		(at 59.69 180.34 0)
@@
 		(effects
 			(font
+				(size 1.27 1.27)
+			)
+			(justify left bottom)
+		)
+	)
+	(label "PB3"
+		(at 386.08 60.96 0)
+		(effects
+			(font

Commit message: esd protection for usb data lines
Parts:
- added D6: USBLC6-2SC6, easyeda2kicad:SOT-23-6_L2.9-W1.6-P0.95-LS2.8-BL, symbol easyeda2kicad:USBLC6-2SC6
- added SB1, SB2: Circuit Breaker, Jumper:SolderJumper-2_P1.3mm_Open_TrianglePad1.0x1.5mm, symbol MCD_TOOLS:root_0_Circuit Breaker_MCD_TOOLS.SCHLIB
Connections:
- net GND: now also D6.2
- net OSC_IN: now also SB2.1
- net OSC_OUT: now also SB1.1
- net PB14: now also D6.1, D6.6
- net PB15: now also D6.3, D6.4
- net PH0: now also SB2.2
- net PH1: now also SB1.2
- no-connect marks 4 -> 5
Other:
- note added: "CC1 and CC2 set to device mode for simplicity, power negotiation unused for USB MICRO AB equivalent is "ID" pin"
- note added: "ESD protection for data lines figure 19 from tcpp01-m12.pdf"
- note added: "GND"
- note added: "I/O1"
- note added: "I/O2"
- note added: "VBUS"
- moved on the sheet: C4, C7, C8, C9, D2, D3, D4, LED1, R1, R27, R29, R4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

Commit message: quick save
Parts:
- removed LED1: FC-2012UGK-520D5, easyeda2kicad:LED0805-R-RD, symbol easyeda2kicad:FC-2012UGK-520D5
- added D5: Red, PCM_JLCPCB:D_0603, symbol PCM_JLCPCB-Diodes:LED,0603,Red
Connections:
- net GND: now also D5.1
- net at R29.2: now also D5.2
- net LED_GREEN renamed LED_RED2
Other:
- note added: "CC1 and CC2 set to device mode for simplicity, dual role device feature unused for USB MICRO AB equivalent is "ID" pin"
- note added: "ESD protection for data lines from figure 19 from tcpp01-m12.pdf"
- note removed: "CC1 and CC2 set to device mode for simplicity, power negotiation unused for USB MICRO AB equivalent is "ID" pin"
- note removed: "ESD protection for data lines figure 19 from tcpp01-m12.pdf"
Changed lines of the file:
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@@
 		)
 	)
-	(text "ESD protection for data lines\nfigure 19 from tcpp01-m12.pdf"
+	(text "ESD protection for data lines\nfrom figure 19 from tcpp01-m12.pdf"
 		(exclude_from_sim no)
 		(at 54.356 266.954 0)
@@
 		)
 	)
-	(text "CC1 and CC2 set to device mode for simplicity, power negotiation unused\nfor USB MICRO AB equivalent is \"ID\" pin"
+	(text "CC1 and CC2 set to device mode for simplicity, dual role device feature unused\nfor USB MICRO AB equivalent is \"ID\" pin"
 		(exclude_from_sim no)
-		(at 112.522 301.498 0)
+		(at 112.522 302.26 0)
 		(effects
 			(font
@@
 	(wire
 		(pts
+			(xy 306.07 160.02) (xy 306.07 161.29)
+		)
+		(stroke
+			(width 0)
+			(type default)
+		)
+	)
+	(wire
+		(pts
 			(xy 82.55 81.28) (xy 80.01 81.28)
 		)
@@
 	(wire
 		(pts
+			(xy 306.07 151.13) (xy 306.07 152.4)
+		)
+		(stroke
+			(width 0)
+			(type default)
+		)
+	)
+	(wire
+		(pts
 			(xy 311.15 -87.63) (xy 321.31 -87.63)
 		)
@@
 		)
 	)
-	(label "LED_GREEN"
+	(label "LED_RED2"
 		(at 176.53 129.54 180)
 		(effects
@@
 		)
 	)
-	(label "LED_GREEN"
+	(label "LED_RED2"
 		(at 306.07 142.24 180)
 		(effects
@@
 	)
 	(symbol
+		(lib_id "PCM_JLCPCB-Diodes:LED,0603,Red")
+		(at 306.07 156.21 0)
+		(unit 1)
+		(exclude_from_sim no)
+		(in_bom yes)
+		(on_board yes)
+		(dnp no)
+		(fields_autoplaced yes)
+		(property "Reference" "D5"
+			(at 308.61 154.8446 0)
+			(effects
+				(font
+					(size 1.27 1.27)
+				)
+				(justify left)
+			)
+		)
+		(property "Value" "Red"
+			(at 308.61 157.3847 0)
+			(effects
+				(font
+					(size 0.8 0.8)
+				)
+				(justify left)
+			)
+		)
+		(property "Footprint" "PCM_JLCPCB:D_0603"
+			(at 304.292 156.21 90)
+			(effects
+				(font
+					(size 1.27 1.27)
+				)
+				(hide yes)
+			)
+		)
+		(property "Datasheet" "https://www.lcsc.com/datasheet/lcsc_datasheet_1810231112_Hubei-KENTO-Elec-KT-0603R_C2286.pdf"
+			(at 306.07 156.21 0)
+			(effects
+				(font
+					(size 1.27 1.27)
+				)
+				(hide yes)
+			)
+		)
+		(property "Description" "-40°C~+85°C Red 0603 LED Indication - Discrete ROHS"
+			(at 306.07 156.21 0)
+			(effects
+				(font
+					(size 1.27 1.27)
+				)
+				(hide yes)
+			)
+		)
+		(property "LCSC" "C2286"
+			(at 306.07 156.21 0)
+			(effects
+				(font
+					(size 1.27 1.27)
+				)
+				(hide yes)
+			)
+		)
+		(property "Stock" "5373336"
+			(at 306.07 156.21 0)
+			(effects
+				(font
+					(size 1.27 1.27)
+				)
+				(hide yes)
+			)
+		)
+		(property "Price" "0.009USD"
+			(at 306.07 156.21 0)
+			(effects
+				(font
+					(size 1.27 1.27)
+				)
+				(hide yes)
+			)
+		)
+		(property "Process" "SMT"
+			(at 306.07 156.21 0)
+			(effects
+				(font
+					(size 1.27 1.27)
+				)
+				(hide yes)
+			)
+		)
+		(property "Minimum Qty" "20"
+			(at 306.07 156.21 0)
+			(effects
+				(font
+					(size 1.27 1.27)
+				)
+				(hide yes)
+			)
+		)
+		(property "Attrition Qty" "10"
+			(at 306.07 156.21 0)
+			(effects
+				(font
+					(size 1.27 1.27)
+				)
+				(hide yes)
+			)
+		)
+		(property "Class" "Basic Component"
+			(at 306.07 156.21 0)
+			(effects
+				(font
+					(size 1.27 1.27)
+				)
+				(hide yes)
+			)
+		)
+		(property "Category" "Optocouplers & LEDs & Infrared,Light Emitting Diodes (LED)"
+			(at 306.07 156.21 0)
+			(effects
+				(font
+					(size 1.27 1.27)
+				)
+				(hide yes)
+			)
+		)
+		(property "Manufacturer" "Hubei KENTO Elec"
+			(at 306.07 156.21 0)
+			(effects
+				(font
+					(size 1.27 1.27)
+				)
+				(hide yes)
+			)
+		)
+		(property "Part" "KT-0603R"
+			(at 306.07 156.21 0)
+			(effects
+				(font
+					(size 1.27 1.27)
+				)
+				(hide yes)
+			)
+		)
+		(pin "1"
+		)
+		(pin "2"
+		)
+		(instances
+			(project "STM32F429ZIT6"
+				(path "/bb5a47a2-47e2-4f6f-8bb5-5479733ff8ef"
+					(reference "D5")
+					(unit 1)
+				)
+			)
+		)
+	)
+	(symbol
 		(lib_id "PCM_JLCPCB-Resistors:0603,47kΩ")
 		(at 304.8 260.35 270)
@@
 					(unit 1)
 				)
-			)
-		)
-	)
-	(symbol
-		(lib_id "easyeda2kicad:FC-2012UGK-520D5")
-		(at 305.05 156.21 90)
-		(unit 1)
-		(exclude_from_sim no)
-		(in_bom yes)
-		(on_board yes)
-		(dnp no)
-		(fields_autoplaced yes)
-		(property "Reference" "LED1"
-			(at 308.86 156.2099 90)
-			(effects
-				(font
-					(size 1.27 1.27)
-				)
-				(justify right)
-			)
-		)
-		(property "Value" "FC-2012UGK-520D5"
-			(at 308.86 158.7499 90)
-			(effects
-				(font
-					(size 1.27 1.27)
-				)
-				(justify right)
-			)
-		)
-		(property "Footprint" "easyeda2kicad:LED0805-R-RD"
-			(at 313.69 156.21 0)
-			(effects
-				(font
-					(size 1.27 1.27)
-				)
-				(hide yes)
-			)
-		)
-		(property "Datasheet" "https://lcsc.com/product-detail/Light-Emitting-Diodes-LED_Emerald-SMDLED-180-330mcd_C84260.html"
-			(at 316.23 156.21 0)
-			(effects
-				(font
-					(size 1.27 1.27)
-				)
-				(hide yes)
-			)
-		)
-		(property "Description" ""
-			(at 305.05 156.21 0)
-			(effects
-				(font
-					(size 1.27 1.27)
-				)
-				(hide yes)
-			)
-		)
-		(property "LCSC Part" "C84260"
-			(at 318.77 156.21 0)
-			(effects
-				(font
-					(size 1.27 1.27)
-				)
-				(hide yes)
-			)
-		)
-		(pin "1"
-		)
-		(pin "2"
-		)
-		(instances
-			(project "STM32F429ZIT6"
-				(path "/bb5a47a2-47e2-4f6f-8bb5-5479733ff8ef"
-					(reference "LED1")
-					(unit 1)
-				)

Commit message: added screen print labels, line in detect need to test
Parts:
- added J1: Conn_01x02_Pin, Connector_PinHeader_2.54mm:PinHeader_1x02_P2.54mm_Vertical, symbol Connector:Conn_01x02_Pin
Connections:
- net 3V is gone; now on net +3.3V: P2.1, P2.2
- net 5V is gone; now on net +3.3V: P1.1, P1.2
- net PC13 is gone; now on net LINEIN_DTCT: P1.12, U.1.7 (PC13)
- net AUXOUT1: now also J1.1 (Pin_1)
- net AUXOUT2: now also J1.2 (Pin_2)
Other:
- note removed: "3V"
- note removed: "5V"

Commit message: measuring trace lengths, looks ok so far! almost done
Parts:
- removed H1, H2, H3, H4: ScrewMount, MountingHole:MountingHole_3.2mm_M3, symbol Mechanical:MountingHole
Connections:
- net +5V: now also P2.63, P2.64
- net GND: no longer P2.63, P2.64
