File: STM32F429ZIT6.kicad_sch (KiCad schematic)
At the start: 117 parts, among them J1 Conn_01x02_Pin, J2 Conn_01x05_Pin, P1 Header 32X2, P2 Header 32X2, SW1 K3-1235S, U2 LD3985M33R, U3 MCP6004, U4 NAU88C22YG_C914209, U5 RCLAMP0521P.TCT_C3029033, U6 RCLAMP0521P.TCT_C3029033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

Commit message: xtal fix
Parts:
- removed C4, C7, C8, C9: 100nF, PCM_JLCPCB:C_0402, symbol PCM_JLCPCB-Capacitors:0402,100nF
Connections:
- net GND: now also X1.2 (GND), X1.4 (GND)
- net OSC_IN: now also C31.1
- net OSC_OUT: now also C30.1
Other:
- note added: "(load-stray)*2 (10-5)*2=10 Osc C load = 10pF Stray 1-5~ per pin need to measure assume 5pf from "Phil's Lab #65" around 30 mins also AN2867 figure 5"
- note removed: "(load-stray)*2 (10-5)*2=10 Osc C load = 10pF Stray 1-5~ per pin need to measure assume 5pf"
- note removed: "3v3 power filtering"
