File: STM32F429ZIT6.kicad_pcb (KiCad board)
At the start: 4 copper layers, 74.9 x 114.5 mm, 123 parts, among them J1 Conn_01x02_Pin, J2 Conn_01x05_Pin, P1 Header 32X2, P2 Header 32X2, SW1 K3-1235S, U2 LD3985M33R, U3 MCP6004, U4 NAU88C22YG_C914209, U5 RCLAMP0521P.TCT_C3029033, U6 RCLAMP0521P.TCT_C3029033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

Commit message: measuring trace lengths, looks ok so far! almost done
Parts:
- removed H1, H2, H3, H4: ScrewMount, MountingHole:MountingHole_3.2mm_M3
- moved D3 22.6 mm to (138.4, 149.4)
- moved R1 22.6 mm to (136.4, 149.4)
- moved C1 1.22 mm to (134.3, 143.4)
- moved C10 1.22 mm to (129.6, 97.4)
- moved C23 1.22 mm to (148.3, 84.7)
- moved C25 1.22 mm to (129.7, 110.2)
- moved C33 1.22 mm to (140.6, 68.7)
- moved C38 1.22 mm to (146.7, 70.7)
- moved C4 1.22 mm to (164.6, 146.3)
- moved C5 1.22 mm to (134.2, 137.6)
- moved C58 1.22 mm to (150.1, 131.5)
- moved C6 1.22 mm to (134.4, 135.9)
- moved D1 1.22 mm to (131.9, 138.1)
- moved D2 1.22 mm to (130.4, 143.6)
- moved D5 1.22 mm to (162.6, 99.2)
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Connections:
- P2 pad 63: GND -> +5V
- P2 pad 64: GND -> +5V
Routing:
- net +5V: track 9.49 -> 10.3 mm, vias 0 -> 1
- added copper zone on In1.Cu, net +5V
Other:
- board size 74.9 x 114.5 mm -> 74.8 x 114.5 mm
- board text added: "5V"
- board text added: "SWCLK"
- board text added: "SWDIO"
- board text added: "SWO"
- board text added: "stm32f429zit6 dev board 8MB sdram & stereo in/out 5/15/26"
- board text removed: "stm32f429zit6 dev board 8MB sdram & stereo audio in/out 5/14/26"

Commit message: xtal fix
Parts:
- removed C4, C7, C8, C9: 100nF, PCM_JLCPCB:C_0402
- moved C31 6.51 mm to (144.8, 83.2)
- moved C30 6.25 mm to (137.9, 83.6), turned to 90 degrees
- moved SB2 1.47 mm to (142.8, 77.9)
- moved SB1 1.25 mm to (140.0, 77.9)
- moved G*** 0.66 mm to (160.1, 141.4)
- moved X1 0.54 mm to (141.4, 83.3)
Connections:
- C30 pad 1: Net-(C30-Pad1) -> /OSC_OUT
- C31 pad 1: Net-(C30-Pad1) -> /OSC_IN
- X1 pad 2: Net-(C30-Pad1) -> GND
- X1 pad 4: Net-(C30-Pad1) -> GND
Routing:
- net Net-(C30-Pad1): track 11.7 -> 0.00 mm
- net /OSC_OUT: track 9.84 -> 14.5 mm, vias 2 -> 0
- net +3.3V: track 82.9 -> 79.1 mm, vias 35 -> 31
- net /OSC_IN: track 11.2 -> 12.9 mm, vias 2 -> 0
- net /PH0: track 32.1 -> 30.9 mm
- net /PH1: track 25.4 -> 24.6 mm
- net GND: track 90.1 -> 90.0 mm, vias 45 -> 46
Other:
- board text removed: "LIN"
- board text removed: "RIN"

Commit message: DONE i think!!!!
Parts:
- moved C30 0.10 mm to (138.0, 83.6)
Routing:
- net GND: track 90.0 -> 88.6 mm, vias 46 -> 47
Other:
- board text added: "stm32f429zit6 dev board 8MB sdram & stereo in/out 5/16/26"
- board text removed: "stm32f429zit6 dev board 8MB sdram & stereo in/out 5/15/26"
Changed lines of the file:
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@@
 	(footprint "PCM_JLCPCB:C_0402"
 		(layer "F.Cu")
-		(at 137.9 83.6 90)
+		(at 138 83.6 90)
 		(descr "Capacitor SMD 0402 (1005 Metric), square (rectangular) end terminal, IPC_7351 nominal, (Body size source: IPC-SM-782 page 76, https://www.pcb-3d.com/wordpress/wp-content/uploads/ipc-sm-782a_amendment_1_and_2.pdf), generated with kicad-footprint-generator")
 		(tags "capacitor")
@@
 		(at 141.4 83.33 180)
 		(property "Reference" "X1"
-			(at 0.99 2.47 0)
+			(at -3.3 2.83 0)
 			(layer "F.SilkS")
 			(effects
@@
 		)
 	)
-	(gr_text "stm32f429zit6 dev board\n8MB sdram & stereo in/out\n5/15/26"
-		(at 142.09 138.45 0)
+	(gr_text "stm32f429zit6 dev board\n8MB sdram & stereo in/out\n5/16/26"
+		(at 142.09 138.7 0)
 		(layer "F.SilkS")
 		(effects
@@
 	)
 	(segment
-		(start 149.19 58.15)
-		(end 148.13 58.15)
-		(width 0.15)
-		(layer "F.Cu")
-		(net 3)
-	)
-	(segment
 		(start 171.13 54.51)
 		(end 171.8 54.51)
@@
 	)
 	(segment
+		(start 139.85 70.65)
+		(end 139.8 70.6)
+		(width 0.15)
+		(layer "F.Cu")
+		(net 3)
+	)
+	(segment
 		(start 171.8 54.51)
 		(end 171.94 54.65)
@@
 	)
 	(segment
-		(start 139.59 70.35)
-		(end 139.54 70.3)
-		(width 0.15)
-		(layer "F.Cu")
-		(net 3)
-	)
-	(segment
 		(start 131.39 146.11125)
 		(end 131.14 146.36125)
@@
 	)
 	(segment
+		(start 140.93 70.65)
+		(end 139.85 70.65)
+		(width 0.15)
+		(layer "F.Cu")
+		(net 3)
+	)
+	(segment
 		(start 125.58 144.92875)
 		(end 124.74 145.76875)
@@
 	)
 	(segment
-		(start 139.89 70.65)
-		(end 139.59 70.35)
-		(width 0.15)
-		(layer "F.Cu")
-		(net 3)
-	)
-	(segment
 		(start 131.49 109.69)
 		(end 131.23 109.95)
@@
 	)
 	(segment
-		(start 140.93 70.65)
-		(end 139.89 70.65)
-		(width 0.15)
-		(layer "F.Cu")
-		(net 3)
-	)
-	(segment
 		(start 150.61 131.455679)
 		(end 151.31 131.455679)
@@
 	)
 	(via
-		(at 138.150202 112.2267)
+		(at 127.3 88.6)
 		(size 0.6)
 		(drill 0.35)
 		(layers "F.Cu" "B.Cu")
+		(free yes)
 		(net 3)
 	)
 	(via
-		(at 163.94 51.8)
+		(at 138.150202 112.2267)
 		(size 0.6)
 		(drill 0.35)
@@
 	)
 	(via
-		(at 154.64 81.62)
+		(at 163.94 51.8)
 		(size 0.6)
 		(drill 0.35)
 		(layers "F.Cu" "B.Cu")
-		(free yes)
 		(net 3)
 	)
 	(via
-		(at 139.59 70.35)
+		(at 154.64 81.62)
 		(size 0.6)
 		(drill 0.35)
 		(layers "F.Cu" "B.Cu")
+		(free yes)
 		(net 3)
 	)
@@
 	)
 	(via
-		(at 149.19 58.15)
+		(at 141 80.6)
 		(size 0.6)
 		(drill 0.35)
 		(layers "F.Cu" "B.Cu")
+		(free yes)
 		(net 3)
 	)
 	(via
-		(at 141 80.6)
+		(at 139.8 70.6)
 		(size 0.6)
 		(drill 0.35)
 		(layers "F.Cu" "B.Cu")
-		(free yes)
 		(net 3)
 	)
@@
 	)
 	(via
-		(at 168.72 54.26)
-		(size 0.6)
-		(drill 0.35)
-		(layers "F.Cu" "B.Cu")
-		(net 3)
-	)
-	(via
 		(at 154.67 87.34)
 		(size 0.6)
@@
 	)
 	(via
+		(at 160.1 87.9)
+		(size 0.6)
+		(drill 0.35)
+		(layers "F.Cu" "B.Cu")
+		(free yes)
+		(net 3)
+	)
+	(via
+		(at 168.72 54.26)
+		(size 0.6)
+		(drill 0.35)
+		(layers "F.Cu" "B.Cu")
+		(net 3)
+	)
+	(via
 		(at 156.49 102.05)
 		(size 0.6)
@@
 	)
 	(segment
-		(start 126.972169 77.276)
-		(end 139.44 89.743831)
+		(start 114.3 76.2)
+		(end 115.6 77.5)
 		(width 0.15)
 		(layer "B.Cu")
@@
 	)
 	(segment
-		(start 114.3 76.2)
-		(end 115.376 77.276)
+		(start 139.44 89.743831)
+		(end 139.44 90.15)
 		(width 0.15)
 		(layer "B.Cu")
@@
 	)
 	(segment
-		(start 115.376 77.276)
-		(end 126.972169 77.276)
+		(start 127.196169 77.5)
+		(end 139.44 89.743831)
 		(width 0.15)
 		(layer "B.Cu")
@@
 	)
 	(segment
-		(start 139.44 89.743831)
-		(end 139.44 90.15)
+		(start 115.6 77.5)
+		(end 127.196169 77.5)
 		(width 0.15)
 		(layer "B.Cu")
@@
 	)
 	(segment
-		(start 119.615678 73.45)
-		(end 118.665678 72.5)
+		(start 139.525 73.9)
+		(end 120.065678 73.9)
 		(width 0.15)
 		(layer "F.Cu")
@@
 	)
 	(segment
-		(start 115.46 72.5)
-		(end 114.3 73.66)
+		(start 142.8 77.175)
+		(end 139.525 73.9)
 		(width 0.15)
 		(layer "F.Cu")
@@
 	)
 	(segment
-		(start 142.8 77.175)
-		(end 139.075 73.45)
+		(start 118.665678 72.5)
+		(end 115.46 72.5)
 		(width 0.15)
 		(layer "F.Cu")
@@
 	)
 	(segment
-		(start 139.075 73.45)
-		(end 119.615678 73.45)
+		(start 120.065678 73.9)
+		(end 118.665678 72.5)
 		(width 0.15)
 		(layer "F.Cu")
@@
 	)
 	(segment
-		(start 118.665678 72.5)
-		(end 115.46 72.5)
+		(start 115.46 72.5)
+		(end 114.3 73.66)
 		(width 0.15)
 		(layer "F.Cu")
