File: docs/mb1075_bdp/MB1075E/Altium_Designer/IO_Peripherals.kicad_sch (KiCad schematic)
At the start: 23 parts

Commit message: save before i break everything out instead idk why i didnt do that
Parts:
- removed C (x3): 100nF, 0402C, symbol MCD_TOOLS:root_1_Capacitor_ST_MCD_TOOLS.SchLib
- removed C: 10nF/25V, 0603C, symbol Miscellaneous Devices:root_1_CAP_Miscellaneous Devices.IntLib
- removed C: 10uF, 0603C, symbol Miscellaneous Devices:root_1_CAP_Miscellaneous Devices.IntLib
- removed LD: Red, 0603D, symbol Miscellaneous Devices:root_0_LED2_Miscellaneous Devices.IntLib
- removed LD: Green, 0603D, symbol Miscellaneous Devices:root_0_LED2_Miscellaneous Devices.IntLib
- removed R: 680, 0603R, symbol MCD_TOOLS:root_0_Resistor_ST_MCD_TOOLS.SchLib
- removed R: 100K, 0402R, symbol MCD_TOOLS:root_1_Resistor_ST_MCD_TOOLS.SchLib
- removed R: 330, 0402R, symbol MCD_TOOLS:root_0_Resistor_ST_MCD_TOOLS.SchLib
- removed R: 100, 0402R, symbol MCD_TOOLS:root_0_Resistor_ST_MCD_TOOLS.SchLib
- removed R: 510, 0603R, symbol MCD_TOOLS:root_0_Resistor_ST_MCD_TOOLS.SchLib
- removed R: 220K, 0402R, symbol MCD_TOOLS:root_1_Resistor_ST_MCD_TOOLS.SchLib
- removed R: 10K, 0402R, symbol MCD_TOOLS:root_1_Resistor_ST_MCD_TOOLS.SchLib
- removed SB (x2): Circuit Breaker, JP2_SMD, symbol MB915:root_0_Circuit Breaker_MB915.SCHLIB
- added C: 10uF, 0603C, symbol Miscellaneous Devices:root_1_CAP_Miscellaneous Devices.IntLib
- added C (x3): 100nF, 0402C, symbol MCD_TOOLS:root_1_Capacitor_ST_MCD_TOOLS.SchLib
- added C: 10nF/25V, 0603C, symbol Miscellaneous Devices:root_1_CAP_Miscellaneous Devices.IntLib
- added LD: Green, 0603D, symbol Miscellaneous Devices:root_0_LED2_Miscellaneous Devices.IntLib
- added LD: Red, 0603D, symbol Miscellaneous Devices:root_0_LED2_Miscellaneous Devices.IntLib
- added R: 100K, 0402R, symbol MCD_TOOLS:root_1_Resistor_ST_MCD_TOOLS.SchLib
- added R: 10K, 0402R, symbol MCD_TOOLS:root_1_Resistor_ST_MCD_TOOLS.SchLib
- added R: 330, 0402R, symbol MCD_TOOLS:root_0_Resistor_ST_MCD_TOOLS.SchLib
- added R: 220K, 0402R, symbol MCD_TOOLS:root_1_Resistor_ST_MCD_TOOLS.SchLib
- added R: 100, 0402R, symbol MCD_TOOLS:root_0_Resistor_ST_MCD_TOOLS.SchLib
- added R: 680, 0603R, symbol MCD_TOOLS:root_0_Resistor_ST_MCD_TOOLS.SchLib
- added R: 510, 0603R, symbol MCD_TOOLS:root_0_Resistor_ST_MCD_TOOLS.SchLib
- added SB (x2): Circuit Breaker, JP2_SMD, symbol MB915:root_0_Circuit Breaker_MB915.SCHLIB
Connections:
- net 3V: now also C.2, C.2
- net GND: now also C.1, C.1, C.1, C.1, LD.2 (K), LD.2 (K), R.1, R.1
- net NRST: now also SB.1
- net PA0: now also SB.1
- net PG13: now also R.1
- net PG14: now also R.1
- net VDD: now also R.2, R.2
- net at B.1, B.4: now also C.2, R.1, SB.2
- net at C.2, U.14 (PLLFILT): now also C.2
- net at B.2, B.3: now also C.1, R.2, R.2
- net at C.1: now also R.2
- new net: LD.1 (A), R.2 (x2)
- new net: R.1, SB.2
- new net: C.2, R.1

Commit message: KILL ME!!!!!!!!!!!
Parts:
- removed C: 10uF, 0603C, symbol Miscellaneous Devices:root_1_CAP_Miscellaneous Devices.IntLib
- removed C (x3): 100nF, 0402C, symbol MCD_TOOLS:root_1_Capacitor_ST_MCD_TOOLS.SchLib
- removed C: 10nF/25V, 0603C, symbol Miscellaneous Devices:root_1_CAP_Miscellaneous Devices.IntLib
- removed LD: Green, 0603D, symbol Miscellaneous Devices:root_0_LED2_Miscellaneous Devices.IntLib
- removed LD: Red, 0603D, symbol Miscellaneous Devices:root_0_LED2_Miscellaneous Devices.IntLib
- removed R: 100K, 0402R, symbol MCD_TOOLS:root_1_Resistor_ST_MCD_TOOLS.SchLib
- removed R: 10K, 0402R, symbol MCD_TOOLS:root_1_Resistor_ST_MCD_TOOLS.SchLib
- removed R: 330, 0402R, symbol MCD_TOOLS:root_0_Resistor_ST_MCD_TOOLS.SchLib
- removed R: 220K, 0402R, symbol MCD_TOOLS:root_1_Resistor_ST_MCD_TOOLS.SchLib
- removed R: 100, 0402R, symbol MCD_TOOLS:root_0_Resistor_ST_MCD_TOOLS.SchLib
- removed R: 680, 0603R, symbol MCD_TOOLS:root_0_Resistor_ST_MCD_TOOLS.SchLib
- removed R: 510, 0603R, symbol MCD_TOOLS:root_0_Resistor_ST_MCD_TOOLS.SchLib
- removed SB (x2): Circuit Breaker, JP2_SMD, symbol MB915:root_0_Circuit Breaker_MB915.SCHLIB
- added C (x3): 100nF, 0402C, symbol MCD_TOOLS:root_1_Capacitor_ST_MCD_TOOLS.SchLib
- added C: 10nF/25V, 0603C, symbol Miscellaneous Devices:root_1_CAP_Miscellaneous Devices.IntLib
- added C: 10uF, 0603C, symbol Miscellaneous Devices:root_1_CAP_Miscellaneous Devices.IntLib
- added LD: Green, 0603D, symbol Miscellaneous Devices:root_0_LED2_Miscellaneous Devices.IntLib
- added LD: Red, 0603D, symbol Miscellaneous Devices:root_0_LED2_Miscellaneous Devices.IntLib
- added R: 10K, 0402R, symbol MCD_TOOLS:root_1_Resistor_ST_MCD_TOOLS.SchLib
- added R: 330, 0402R, symbol MCD_TOOLS:root_0_Resistor_ST_MCD_TOOLS.SchLib
- added R: 220K, 0402R, symbol MCD_TOOLS:root_1_Resistor_ST_MCD_TOOLS.SchLib
- added R: 510, 0603R, symbol MCD_TOOLS:root_0_Resistor_ST_MCD_TOOLS.SchLib
- added R: 100K, 0402R, symbol MCD_TOOLS:root_1_Resistor_ST_MCD_TOOLS.SchLib
- added R: 100, 0402R, symbol MCD_TOOLS:root_0_Resistor_ST_MCD_TOOLS.SchLib
- added R: 680, 0603R, symbol MCD_TOOLS:root_0_Resistor_ST_MCD_TOOLS.SchLib
- added SB (x2): Circuit Breaker, JP2_SMD, symbol MB915:root_0_Circuit Breaker_MB915.SCHLIB
Connections:
- net 3V: now also C.2, C.2
- net GND: now also C.1, C.1, C.1, C.1, LD.2 (K), LD.2 (K), R.1, R.1
- net NRST: now also SB.1
- net PA0: now also SB.1
- net PG13: now also R.1
- net PG14: now also R.1
- net VDD: now also R.2, R.2
- net at B.1, B.4: now also C.2, R.1, SB.2
- net at C.1: now also R.2
- net at B.2, B.3: now also C.1, R.2, R.2
- net at C.2, U.14 (PLLFILT): now also C.2
- new net: LD.1 (A), R.2 (x2)
- new net: C.2, R.1
- new net: R.1, SB.2

Commit message: esd protection for usb data lines
Parts:
- removed C (x3): 100nF, 0402C, symbol MCD_TOOLS:root_1_Capacitor_ST_MCD_TOOLS.SchLib
- removed C: 10nF/25V, 0603C, symbol Miscellaneous Devices:root_1_CAP_Miscellaneous Devices.IntLib
- removed C: 10uF, 0603C, symbol Miscellaneous Devices:root_1_CAP_Miscellaneous Devices.IntLib
- removed LD: Green, 0603D, symbol Miscellaneous Devices:root_0_LED2_Miscellaneous Devices.IntLib
- removed LD: Red, 0603D, symbol Miscellaneous Devices:root_0_LED2_Miscellaneous Devices.IntLib
- removed R: 10K, 0402R, symbol MCD_TOOLS:root_1_Resistor_ST_MCD_TOOLS.SchLib
- removed R: 330, 0402R, symbol MCD_TOOLS:root_0_Resistor_ST_MCD_TOOLS.SchLib
- removed R: 220K, 0402R, symbol MCD_TOOLS:root_1_Resistor_ST_MCD_TOOLS.SchLib
- removed R: 510, 0603R, symbol MCD_TOOLS:root_0_Resistor_ST_MCD_TOOLS.SchLib
- removed R: 100K, 0402R, symbol MCD_TOOLS:root_1_Resistor_ST_MCD_TOOLS.SchLib
- removed R: 100, 0402R, symbol MCD_TOOLS:root_0_Resistor_ST_MCD_TOOLS.SchLib
- removed R: 680, 0603R, symbol MCD_TOOLS:root_0_Resistor_ST_MCD_TOOLS.SchLib
- removed SB (x2): Circuit Breaker, JP2_SMD, symbol MB915:root_0_Circuit Breaker_MB915.SCHLIB
- added C: 10nF/25V, 0603C, symbol Miscellaneous Devices:root_1_CAP_Miscellaneous Devices.IntLib
- added C (x3): 100nF, 0402C, symbol MCD_TOOLS:root_1_Capacitor_ST_MCD_TOOLS.SchLib
- added C: 10uF, 0603C, symbol Miscellaneous Devices:root_1_CAP_Miscellaneous Devices.IntLib
- added LD: Green, 0603D, symbol Miscellaneous Devices:root_0_LED2_Miscellaneous Devices.IntLib
- added LD: Red, 0603D, symbol Miscellaneous Devices:root_0_LED2_Miscellaneous Devices.IntLib
- added R: 100K, 0402R, symbol MCD_TOOLS:root_1_Resistor_ST_MCD_TOOLS.SchLib
- added R: 220K, 0402R, symbol MCD_TOOLS:root_1_Resistor_ST_MCD_TOOLS.SchLib
- added R: 510, 0603R, symbol MCD_TOOLS:root_0_Resistor_ST_MCD_TOOLS.SchLib
- added R: 10K, 0402R, symbol MCD_TOOLS:root_1_Resistor_ST_MCD_TOOLS.SchLib
- added R: 330, 0402R, symbol MCD_TOOLS:root_0_Resistor_ST_MCD_TOOLS.SchLib
- added R: 680, 0603R, symbol MCD_TOOLS:root_0_Resistor_ST_MCD_TOOLS.SchLib
- added R: 100, 0402R, symbol MCD_TOOLS:root_0_Resistor_ST_MCD_TOOLS.SchLib
- added SB (x2): Circuit Breaker, JP2_SMD, symbol MB915:root_0_Circuit Breaker_MB915.SCHLIB
Connections:
- net 3V: now also C.2, C.2
- net GND: now also C.1, C.1, C.1, C.1, LD.2 (K), LD.2 (K), R.1, R.1
- net NRST: now also SB.1
- net PA0: now also SB.1
- net PG13: now also R.1
- net PG14: now also R.1
- net VDD: now also R.2, R.2
- net at B.1, B.4: now also C.2, R.1, SB.2
- net at B.2, B.3: now also C.1, R.2, R.2
- net at C.1: now also R.2
- net at C.2, U.14 (PLLFILT): now also C.2
- new net: R.1, SB.2
- new net: LD.1 (A), R.2 (x2)
- new net: C.2, R.1

Commit message: measuring trace lengths, looks ok so far! almost done
Parts:
- removed C: 10nF/25V, 0603C, symbol Miscellaneous Devices:root_1_CAP_Miscellaneous Devices.IntLib
- removed C (x3): 100nF, 0402C, symbol MCD_TOOLS:root_1_Capacitor_ST_MCD_TOOLS.SchLib
- removed C: 10uF, 0603C, symbol Miscellaneous Devices:root_1_CAP_Miscellaneous Devices.IntLib
- removed LD: Green, 0603D, symbol Miscellaneous Devices:root_0_LED2_Miscellaneous Devices.IntLib
- removed LD: Red, 0603D, symbol Miscellaneous Devices:root_0_LED2_Miscellaneous Devices.IntLib
- removed R: 100K, 0402R, symbol MCD_TOOLS:root_1_Resistor_ST_MCD_TOOLS.SchLib
- removed R: 220K, 0402R, symbol MCD_TOOLS:root_1_Resistor_ST_MCD_TOOLS.SchLib
- removed R: 510, 0603R, symbol MCD_TOOLS:root_0_Resistor_ST_MCD_TOOLS.SchLib
- removed R: 10K, 0402R, symbol MCD_TOOLS:root_1_Resistor_ST_MCD_TOOLS.SchLib
- removed R: 330, 0402R, symbol MCD_TOOLS:root_0_Resistor_ST_MCD_TOOLS.SchLib
- removed R: 680, 0603R, symbol MCD_TOOLS:root_0_Resistor_ST_MCD_TOOLS.SchLib
- removed R: 100, 0402R, symbol MCD_TOOLS:root_0_Resistor_ST_MCD_TOOLS.SchLib
- removed SB (x2): Circuit Breaker, JP2_SMD, symbol MB915:root_0_Circuit Breaker_MB915.SCHLIB
- added C: 10uF, 0603C, symbol Miscellaneous Devices:root_1_CAP_Miscellaneous Devices.IntLib
- added C: 10nF/25V, 0603C, symbol Miscellaneous Devices:root_1_CAP_Miscellaneous Devices.IntLib
- added C (x3): 100nF, 0402C, symbol MCD_TOOLS:root_1_Capacitor_ST_MCD_TOOLS.SchLib
- added LD: Red, 0603D, symbol Miscellaneous Devices:root_0_LED2_Miscellaneous Devices.IntLib
- added LD: Green, 0603D, symbol Miscellaneous Devices:root_0_LED2_Miscellaneous Devices.IntLib
- added R: 220K, 0402R, symbol MCD_TOOLS:root_1_Resistor_ST_MCD_TOOLS.SchLib
- added R: 100K, 0402R, symbol MCD_TOOLS:root_1_Resistor_ST_MCD_TOOLS.SchLib
- added R: 100, 0402R, symbol MCD_TOOLS:root_0_Resistor_ST_MCD_TOOLS.SchLib
- added R: 510, 0603R, symbol MCD_TOOLS:root_0_Resistor_ST_MCD_TOOLS.SchLib
- added R: 330, 0402R, symbol MCD_TOOLS:root_0_Resistor_ST_MCD_TOOLS.SchLib
- added R: 10K, 0402R, symbol MCD_TOOLS:root_1_Resistor_ST_MCD_TOOLS.SchLib
- added R: 680, 0603R, symbol MCD_TOOLS:root_0_Resistor_ST_MCD_TOOLS.SchLib
- added SB (x2): Circuit Breaker, JP2_SMD, symbol MB915:root_0_Circuit Breaker_MB915.SCHLIB
Connections:
- net 3V: now also C.2, C.2
- net GND: now also C.1, C.1, C.1, C.1, LD.2 (K), LD.2 (K), R.1, R.1
- net NRST: now also SB.1
- net PA0: now also SB.1
- net PG13: now also R.1
- net PG14: now also R.1
- net VDD: now also R.2, R.2
- net at B.2, B.3: now also C.1, R.2, R.2
- net at C.2, U.14 (PLLFILT): now also C.2
- net at B.1, B.4: now also C.2, R.1, SB.2
- net at C.1: now also R.2
- new net: C.2, R.1
- new net: LD.1 (A), R.2 (x2)
- new net: R.1, SB.2
