File: docs/mb1075_bdp/MB1075E/Altium_Designer/LCD-24.kicad_sch (KiCad schematic)
At the start: 34 parts

Commit message: save before i break everything out instead idk why i didnt do that
Parts:
- removed C (x2): 100nF, 0402C, symbol MCD_TOOLS:root_1_Capacitor_ST_MCD_TOOLS.SchLib
- removed R (x11): 4K7, 0402R, symbol MCD_TOOLS:root_1_Resistor_ST_MCD_TOOLS.SchLib
- removed R: [N/A], 0402R, symbol MCD_TOOLS:root_0_Resistor_ST_MCD_TOOLS.SchLib
- removed R (x4): [N/A], 0402R, symbol MCD_TOOLS:root_1_Resistor_ST_MCD_TOOLS.SchLib
- removed R (x2): 0, 0402R, symbol MCD_TOOLS:root_0_Resistor_ST_MCD_TOOLS.SchLib
- removed R (x4): 100K, 0402R, symbol MCD_TOOLS:root_0_Resistor_ST_MCD_TOOLS.SchLib
- removed R: 4K7, 0402R, symbol MCD_TOOLS:root_0_Resistor_ST_MCD_TOOLS.SchLib
- removed R (x4): 0, 0603R, symbol MCD_TOOLS:root_0_Resistor_ST_MCD_TOOLS.SchLib
- added C (x2): 100nF, 0402C, symbol MCD_TOOLS:root_1_Capacitor_ST_MCD_TOOLS.SchLib
- added R (x11): 4K7, 0402R, symbol MCD_TOOLS:root_1_Resistor_ST_MCD_TOOLS.SchLib
- added R (x4): 0, 0603R, symbol MCD_TOOLS:root_0_Resistor_ST_MCD_TOOLS.SchLib
- added R (x4): 100K, 0402R, symbol MCD_TOOLS:root_0_Resistor_ST_MCD_TOOLS.SchLib
- added R (x2): 0, 0402R, symbol MCD_TOOLS:root_0_Resistor_ST_MCD_TOOLS.SchLib
- added R: 4K7, 0402R, symbol MCD_TOOLS:root_0_Resistor_ST_MCD_TOOLS.SchLib
- added R (x4): [N/A], 0402R, symbol MCD_TOOLS:root_1_Resistor_ST_MCD_TOOLS.SchLib
- added R: [N/A], 0402R, symbol MCD_TOOLS:root_0_Resistor_ST_MCD_TOOLS.SchLib
Connections:
- net 3V: now also C.2, C.2, R.1, R.1, R.2, R.2, R.2, R.2, R.2, R.2, R.2
- net ADR_A0: now also R.2, R.2
- net DOTCLK: now also R.1
- net ENABLE: now also R.1
- net GND: now also C.1, C.1, R.1, R.1, R.1, R.1, R.1, R.1, R.1, R.1, R.1, R.1, R.2, R.2, R.2, R.2, R.2
- net HSYNC: now also R.1
- net I2C3_SCL: now also R.1
- net I2C3_SDA: now also R.1
- net IM0: now also R.1, R.2
- net IM1: now also R.1, R.2
- net IM2: now also R.1, R.2
- net IM3: now also R.1, R.2
- net TP_INT1: now also R.1
- net VDD: now also R.2, R.2, R.2
- net VSYNC: now also R.1
- net at CN.45 (LEDK1): now also R.2
- net at CN.46 (LEDK2): now also R.2
- net at CN.47 (LEDK3): now also R.2
- net at CN.48 (LEDK4): now also R.2
- net at U.12 (AUX): now also R.2
- net at U.8 (IN0): now also R.1
- net at U.7 (Data_in): now also R.2
- net at U.9 (IN1): now also R.1
- net at U.12 (IN3): now also R.1
- net at U.11 (IN2): now also R.1

Commit message: KILL ME!!!!!!!!!!!
Parts:
- removed C (x2): 100nF, 0402C, symbol MCD_TOOLS:root_1_Capacitor_ST_MCD_TOOLS.SchLib
- removed R (x11): 4K7, 0402R, symbol MCD_TOOLS:root_1_Resistor_ST_MCD_TOOLS.SchLib
- removed R (x4): 0, 0603R, symbol MCD_TOOLS:root_0_Resistor_ST_MCD_TOOLS.SchLib
- removed R (x4): 100K, 0402R, symbol MCD_TOOLS:root_0_Resistor_ST_MCD_TOOLS.SchLib
- removed R (x2): 0, 0402R, symbol MCD_TOOLS:root_0_Resistor_ST_MCD_TOOLS.SchLib
- removed R: 4K7, 0402R, symbol MCD_TOOLS:root_0_Resistor_ST_MCD_TOOLS.SchLib
- removed R (x4): [N/A], 0402R, symbol MCD_TOOLS:root_1_Resistor_ST_MCD_TOOLS.SchLib
- removed R: [N/A], 0402R, symbol MCD_TOOLS:root_0_Resistor_ST_MCD_TOOLS.SchLib
- added C (x2): 100nF, 0402C, symbol MCD_TOOLS:root_1_Capacitor_ST_MCD_TOOLS.SchLib
- added R (x11): 4K7, 0402R, symbol MCD_TOOLS:root_1_Resistor_ST_MCD_TOOLS.SchLib
- added R (x4): [N/A], 0402R, symbol MCD_TOOLS:root_1_Resistor_ST_MCD_TOOLS.SchLib
- added R: [N/A], 0402R, symbol MCD_TOOLS:root_0_Resistor_ST_MCD_TOOLS.SchLib
- added R (x4): 100K, 0402R, symbol MCD_TOOLS:root_0_Resistor_ST_MCD_TOOLS.SchLib
- added R (x2): 0, 0402R, symbol MCD_TOOLS:root_0_Resistor_ST_MCD_TOOLS.SchLib
- added R: 4K7, 0402R, symbol MCD_TOOLS:root_0_Resistor_ST_MCD_TOOLS.SchLib
- added R (x4): 0, 0603R, symbol MCD_TOOLS:root_0_Resistor_ST_MCD_TOOLS.SchLib
Connections:
- net 3V: now also C.2, C.2, R.1, R.1, R.2, R.2, R.2, R.2, R.2, R.2, R.2
- net ADR_A0: now also R.2, R.2
- net DOTCLK: now also R.1
- net ENABLE: now also R.1
- net GND: now also C.1, C.1, R.1, R.1, R.1, R.1, R.1, R.1, R.1, R.1, R.1, R.1, R.2, R.2, R.2, R.2, R.2
- net HSYNC: now also R.1
- net I2C3_SCL: now also R.1
- net I2C3_SDA: now also R.1
- net IM0: now also R.1, R.2
- net IM1: now also R.1, R.2
- net IM2: now also R.1, R.2
- net IM3: now also R.1, R.2
- net TP_INT1: now also R.1
- net VDD: now also R.2, R.2, R.2
- net VSYNC: now also R.1
- net at CN.46 (LEDK2): now also R.2
- net at CN.47 (LEDK3): now also R.2
- net at U.9 (IN1): now also R.1
- net at CN.45 (LEDK1): now also R.2
- net at CN.48 (LEDK4): now also R.2
- net at U.11 (IN2): now also R.1
- net at U.12 (AUX): now also R.2
- net at U.12 (IN3): now also R.1
- net at U.7 (Data_in): now also R.2
- net at U.8 (IN0): now also R.1

Commit message: esd protection for usb data lines
Parts:
- removed C (x2): 100nF, 0402C, symbol MCD_TOOLS:root_1_Capacitor_ST_MCD_TOOLS.SchLib
- removed R (x11): 4K7, 0402R, symbol MCD_TOOLS:root_1_Resistor_ST_MCD_TOOLS.SchLib
- removed R (x4): [N/A], 0402R, symbol MCD_TOOLS:root_1_Resistor_ST_MCD_TOOLS.SchLib
- removed R: [N/A], 0402R, symbol MCD_TOOLS:root_0_Resistor_ST_MCD_TOOLS.SchLib
- removed R (x4): 100K, 0402R, symbol MCD_TOOLS:root_0_Resistor_ST_MCD_TOOLS.SchLib
- removed R (x2): 0, 0402R, symbol MCD_TOOLS:root_0_Resistor_ST_MCD_TOOLS.SchLib
- removed R: 4K7, 0402R, symbol MCD_TOOLS:root_0_Resistor_ST_MCD_TOOLS.SchLib
- removed R (x4): 0, 0603R, symbol MCD_TOOLS:root_0_Resistor_ST_MCD_TOOLS.SchLib
- added C (x2): 100nF, 0402C, symbol MCD_TOOLS:root_1_Capacitor_ST_MCD_TOOLS.SchLib
- added R (x11): 4K7, 0402R, symbol MCD_TOOLS:root_1_Resistor_ST_MCD_TOOLS.SchLib
- added R (x4): 100K, 0402R, symbol MCD_TOOLS:root_0_Resistor_ST_MCD_TOOLS.SchLib
- added R (x2): 0, 0402R, symbol MCD_TOOLS:root_0_Resistor_ST_MCD_TOOLS.SchLib
- added R (x4): 0, 0603R, symbol MCD_TOOLS:root_0_Resistor_ST_MCD_TOOLS.SchLib
- added R: 4K7, 0402R, symbol MCD_TOOLS:root_0_Resistor_ST_MCD_TOOLS.SchLib
- added R (x4): [N/A], 0402R, symbol MCD_TOOLS:root_1_Resistor_ST_MCD_TOOLS.SchLib
- added R: [N/A], 0402R, symbol MCD_TOOLS:root_0_Resistor_ST_MCD_TOOLS.SchLib
Connections:
- net 3V: now also C.2, C.2, R.1, R.1, R.2, R.2, R.2, R.2, R.2, R.2, R.2
- net ADR_A0: now also R.2, R.2
- net DOTCLK: now also R.1
- net ENABLE: now also R.1
- net GND: now also C.1, C.1, R.1, R.1, R.1, R.1, R.1, R.1, R.1, R.1, R.1, R.1, R.2, R.2, R.2, R.2, R.2
- net HSYNC: now also R.1
- net I2C3_SCL: now also R.1
- net I2C3_SDA: now also R.1
- net IM0: now also R.1, R.2
- net IM1: now also R.1, R.2
- net IM2: now also R.1, R.2
- net IM3: now also R.1, R.2
- net TP_INT1: now also R.1
- net VDD: now also R.2, R.2, R.2
- net VSYNC: now also R.1
- net at U.11 (IN2): now also R.1
- net at U.12 (IN3): now also R.1
- net at U.7 (Data_in): now also R.2
- net at U.8 (IN0): now also R.1
- net at U.9 (IN1): now also R.1
- net at CN.48 (LEDK4): now also R.2
- net at CN.45 (LEDK1): now also R.2
- net at CN.46 (LEDK2): now also R.2
- net at CN.47 (LEDK3): now also R.2
- net at U.12 (AUX): now also R.2

Commit message: measuring trace lengths, looks ok so far! almost done
Parts:
- removed C (x2): 100nF, 0402C, symbol MCD_TOOLS:root_1_Capacitor_ST_MCD_TOOLS.SchLib
- removed R (x11): 4K7, 0402R, symbol MCD_TOOLS:root_1_Resistor_ST_MCD_TOOLS.SchLib
- removed R (x4): 100K, 0402R, symbol MCD_TOOLS:root_0_Resistor_ST_MCD_TOOLS.SchLib
- removed R (x2): 0, 0402R, symbol MCD_TOOLS:root_0_Resistor_ST_MCD_TOOLS.SchLib
- removed R (x4): 0, 0603R, symbol MCD_TOOLS:root_0_Resistor_ST_MCD_TOOLS.SchLib
- removed R: 4K7, 0402R, symbol MCD_TOOLS:root_0_Resistor_ST_MCD_TOOLS.SchLib
- removed R (x4): [N/A], 0402R, symbol MCD_TOOLS:root_1_Resistor_ST_MCD_TOOLS.SchLib
- removed R: [N/A], 0402R, symbol MCD_TOOLS:root_0_Resistor_ST_MCD_TOOLS.SchLib
- added C (x2): 100nF, 0402C, symbol MCD_TOOLS:root_1_Capacitor_ST_MCD_TOOLS.SchLib
- added R (x11): 4K7, 0402R, symbol MCD_TOOLS:root_1_Resistor_ST_MCD_TOOLS.SchLib
- added R (x2): 0, 0402R, symbol MCD_TOOLS:root_0_Resistor_ST_MCD_TOOLS.SchLib
- added R (x4): 0, 0603R, symbol MCD_TOOLS:root_0_Resistor_ST_MCD_TOOLS.SchLib
- added R (x4): 100K, 0402R, symbol MCD_TOOLS:root_0_Resistor_ST_MCD_TOOLS.SchLib
- added R (x4): [N/A], 0402R, symbol MCD_TOOLS:root_1_Resistor_ST_MCD_TOOLS.SchLib
- added R: [N/A], 0402R, symbol MCD_TOOLS:root_0_Resistor_ST_MCD_TOOLS.SchLib
- added R: 4K7, 0402R, symbol MCD_TOOLS:root_0_Resistor_ST_MCD_TOOLS.SchLib
Connections:
- net 3V: now also C.2, C.2, R.1, R.1, R.2, R.2, R.2, R.2, R.2, R.2, R.2
- net ADR_A0: now also R.2, R.2
- net DOTCLK: now also R.1
- net ENABLE: now also R.1
- net GND: now also C.1, C.1, R.1, R.1, R.1, R.1, R.1, R.1, R.1, R.1, R.1, R.1, R.2, R.2, R.2, R.2, R.2
- net HSYNC: now also R.1
- net I2C3_SCL: now also R.1
- net I2C3_SDA: now also R.1
- net IM0: now also R.1, R.2
- net IM1: now also R.1, R.2
- net IM2: now also R.1, R.2
- net IM3: now also R.1, R.2
- net TP_INT1: now also R.1
- net VDD: now also R.2, R.2, R.2
- net VSYNC: now also R.1
- net at U.8 (IN0): now also R.1
- net at U.12 (AUX): now also R.2
- net at CN.45 (LEDK1): now also R.2
- net at U.11 (IN2): now also R.1
- net at CN.46 (LEDK2): now also R.2
- net at U.7 (Data_in): now also R.2
- net at CN.47 (LEDK3): now also R.2
- net at CN.48 (LEDK4): now also R.2
- net at U.12 (IN3): now also R.1
- net at U.9 (IN1): now also R.1
