File: docs/mb1075_bdp/MB1075E/Altium_Designer/SDRAM.kicad_sch (KiCad schematic)
At the start: 8 parts, among them U6 IS42S16400J

Commit message: save before i break everything out instead idk why i didnt do that
Parts:
- removed C10, C15, C22, C50, C51, C7, C8: 100nF, 0402C, symbol MCD_TOOLS:U_SDRAM_1_Capacitor_ST_MCD_TOOLS.SchLib
- removed U6: IS42S16400J, TSOP54-II, symbol MCD_TOOLS:U_SDRAM_0_IS45S16400J_MCD_TOOLS.SchLib
- added C (x7): 100nF, 0402C, symbol MCD_TOOLS:root_1_Capacitor_ST_MCD_TOOLS.SchLib
- added U: IS42S16400J, TSOP54-II, symbol MCD_TOOLS:root_0_IS45S16400J_MCD_TOOLS.SchLib
Connections:
- net 3V: now also C.2, C.2, C.2, C.2, C.2, C.2, C.2, U.1 (VDD), U.14 (VDD), U.27 (VDD), U.3 (VDDQ), U.43 (VDDQ), U.49 (VDDQ), U.9 (VDDQ)
- net A0: now also U.23 (A0)
- net A1: now also U.24 (A1)
- net A10: now also U.22 (A10)
- net A11: now also U.35 (A11)
- net A2: now also U.25 (A2)
- net A3: now also U.26 (A3)
- net A4: now also U.29 (A4)
- net A5: now also U.30 (A5)
- net A6: now also U.31 (A6)
- net A7: now also U.32 (A7)
- net A8: now also U.33 (A8)
- net A9: now also U.34 (A9)
- net BA0: now also U.20 (BA0)
- net BA1: now also U.21 (BA1)
- net D0: now also U.2 (DQ0)
- net D1: now also U.4 (DQ1)
- net D10: now also U.45 (DQ10)
- net D11: now also U.47 (DQ11)
- net D12: now also U.48 (DQ12)
- net D13: now also U.50 (DQ13)
- net D14: now also U.51 (DQ14)
- net D15: now also U.53 (DQ15)
- net D2: now also U.5 (DQ2)
- net D3: now also U.7 (DQ3)
- net D4: now also U.8 (DQ4)
- net D5: now also U.10 (DQ5)
- net D6: now also U.11 (DQ6)
- net D7: now also U.13 (DQ7)
- net D8: now also U.42 (DQ8)
- net D9: now also U.44 (DQ9)
- net GND: now also C.1, C.1, C.1, C.1, C.1, C.1, C.1, U.12 (GNDQ), U.28 (GND), U.41 (GND), U.46 (GNDQ), U.52 (GNDQ), U.54 (GND), U.6 (GNDQ)
- net NBL0: now also U.15 (LDQM)
- net NBL1: now also U.39 (UDQM)
- net SDCKE1: now also U.37 (CKE)
- net SDCLK: now also U.38 (CLK)
- net SDNCAS: now also U.17 (~{CAS})
- net SDNE1: now also U.19 (~{CS})
- net SDNRAS: now also U.18 (~{RAS})
- net SDNWE: now also U.16 (~{WE})

Commit message: KILL ME!!!!!!!!!!!
Parts:
- removed C (x7): 100nF, 0402C, symbol MCD_TOOLS:root_1_Capacitor_ST_MCD_TOOLS.SchLib
- removed U: IS42S16400J, TSOP54-II, symbol MCD_TOOLS:root_0_IS45S16400J_MCD_TOOLS.SchLib
- added C10, C15, C22, C50, C51, C7, C8: 100nF, 0402C, symbol MCD_TOOLS:U_SDRAM_1_Capacitor_ST_MCD_TOOLS.SchLib
- added U6: IS42S16400J, TSOP54-II, symbol MCD_TOOLS:U_SDRAM_0_IS45S16400J_MCD_TOOLS.SchLib
Connections:
- net 3V: now also C10.2, C15.2, C22.2, C50.2, C51.2, C7.2, C8.2, U6.1 (VDD), U6.14 (VDD), U6.27 (VDD), U6.3 (VDDQ), U6.43 (VDDQ), U6.49 (VDDQ), U6.9 (VDDQ)
- net A0: now also U6.23 (A0)
- net A1: now also U6.24 (A1)
- net A10: now also U6.22 (A10)
- net A11: now also U6.35 (A11)
- net A2: now also U6.25 (A2)
- net A3: now also U6.26 (A3)
- net A4: now also U6.29 (A4)
- net A5: now also U6.30 (A5)
- net A6: now also U6.31 (A6)
- net A7: now also U6.32 (A7)
- net A8: now also U6.33 (A8)
- net A9: now also U6.34 (A9)
- net BA0: now also U6.20 (BA0)
- net BA1: now also U6.21 (BA1)
- net D0: now also U6.2 (DQ0)
- net D1: now also U6.4 (DQ1)
- net D10: now also U6.45 (DQ10)
- net D11: now also U6.47 (DQ11)
- net D12: now also U6.48 (DQ12)
- net D13: now also U6.50 (DQ13)
- net D14: now also U6.51 (DQ14)
- net D15: now also U6.53 (DQ15)
- net D2: now also U6.5 (DQ2)
- net D3: now also U6.7 (DQ3)
- net D4: now also U6.8 (DQ4)
- net D5: now also U6.10 (DQ5)
- net D6: now also U6.11 (DQ6)
- net D7: now also U6.13 (DQ7)
- net D8: now also U6.42 (DQ8)
- net D9: now also U6.44 (DQ9)
- net GND: now also C10.1, C15.1, C22.1, C50.1, C51.1, C7.1, C8.1, U6.12 (GNDQ), U6.28 (GND), U6.41 (GND), U6.46 (GNDQ), U6.52 (GNDQ), U6.54 (GND), U6.6 (GNDQ)
- net NBL0: now also U6.15 (LDQM)
- net NBL1: now also U6.39 (UDQM)
- net SDCKE1: now also U6.37 (CKE)
- net SDCLK: now also U6.38 (CLK)
- net SDNCAS: now also U6.17 (~{CAS})
- net SDNE1: now also U6.19 (~{CS})
- net SDNRAS: now also U6.18 (~{RAS})
- net SDNWE: now also U6.16 (~{WE})

Commit message: esd protection for usb data lines
Parts:
- removed C10, C15, C22, C50, C51, C7, C8: 100nF, 0402C, symbol MCD_TOOLS:U_SDRAM_1_Capacitor_ST_MCD_TOOLS.SchLib
- removed U6: IS42S16400J, TSOP54-II, symbol MCD_TOOLS:U_SDRAM_0_IS45S16400J_MCD_TOOLS.SchLib
- added C (x7): 100nF, 0402C, symbol MCD_TOOLS:root_1_Capacitor_ST_MCD_TOOLS.SchLib
- added U: IS42S16400J, TSOP54-II, symbol MCD_TOOLS:root_0_IS45S16400J_MCD_TOOLS.SchLib
Connections:
- net 3V: now also C.2, C.2, C.2, C.2, C.2, C.2, C.2, U.1 (VDD), U.14 (VDD), U.27 (VDD), U.3 (VDDQ), U.43 (VDDQ), U.49 (VDDQ), U.9 (VDDQ)
- net A0: now also U.23 (A0)
- net A1: now also U.24 (A1)
- net A10: now also U.22 (A10)
- net A11: now also U.35 (A11)
- net A2: now also U.25 (A2)
- net A3: now also U.26 (A3)
- net A4: now also U.29 (A4)
- net A5: now also U.30 (A5)
- net A6: now also U.31 (A6)
- net A7: now also U.32 (A7)
- net A8: now also U.33 (A8)
- net A9: now also U.34 (A9)
- net BA0: now also U.20 (BA0)
- net BA1: now also U.21 (BA1)
- net D0: now also U.2 (DQ0)
- net D1: now also U.4 (DQ1)
- net D10: now also U.45 (DQ10)
- net D11: now also U.47 (DQ11)
- net D12: now also U.48 (DQ12)
- net D13: now also U.50 (DQ13)
- net D14: now also U.51 (DQ14)
- net D15: now also U.53 (DQ15)
- net D2: now also U.5 (DQ2)
- net D3: now also U.7 (DQ3)
- net D4: now also U.8 (DQ4)
- net D5: now also U.10 (DQ5)
- net D6: now also U.11 (DQ6)
- net D7: now also U.13 (DQ7)
- net D8: now also U.42 (DQ8)
- net D9: now also U.44 (DQ9)
- net GND: now also C.1, C.1, C.1, C.1, C.1, C.1, C.1, U.12 (GNDQ), U.28 (GND), U.41 (GND), U.46 (GNDQ), U.52 (GNDQ), U.54 (GND), U.6 (GNDQ)
- net NBL0: now also U.15 (LDQM)
- net NBL1: now also U.39 (UDQM)
- net SDCKE1: now also U.37 (CKE)
- net SDCLK: now also U.38 (CLK)
- net SDNCAS: now also U.17 (~{CAS})
- net SDNE1: now also U.19 (~{CS})
- net SDNRAS: now also U.18 (~{RAS})
- net SDNWE: now also U.16 (~{WE})

Commit message: measuring trace lengths, looks ok so far! almost done
Parts:
- removed C (x7): 100nF, 0402C, symbol MCD_TOOLS:root_1_Capacitor_ST_MCD_TOOLS.SchLib
- added C (x7): 100nF, 0402C, symbol MCD_TOOLS:root_1_Capacitor_ST_MCD_TOOLS.SchLib
Connections:
- net 3V: now also C.2, C.2, C.2, C.2, C.2, C.2, C.2
- net GND: now also C.1, C.1, C.1, C.1, C.1, C.1, C.1
