File: docs/mb1075_bdp/MB1075E/Altium_Designer/STM32Fx.kicad_sch (KiCad schematic)
At the start: 46 parts, among them U5 STM32F429ZIT6, X2 MC306-G-06Q-32.768, X3 8MHz

Commit message: save before i break everything out instead idk why i didnt do that
Parts:
- removed C20, C21: 20pF, 0402C, symbol MCD_TOOLS:U_STM32Fx_0_Capacitor_ST_MCD_TOOLS.SchLib
- removed C23, C24: 6.8pF, 0402C, symbol MCD_TOOLS:U_STM32Fx_0_Capacitor_ST_MCD_TOOLS.SchLib
- removed C25: 1uF, TAN-A, symbol Miscellaneous Devices:U_STM32Fx_1_Cap Pol1_Miscellaneous Devices.IntLib
- removed C26: 1uF, TAN-A, symbol Miscellaneous Devices:U_STM32Fx_3_Cap Pol1_Miscellaneous Devices.IntLib
- removed C28: 1uF, 0603C, symbol MCD_TOOLS:U_STM32Fx_0_Capacitor_ST_MCD_TOOLS.SchLib
- removed C29, C30, C31, C32, C33, C34, C35, C36, C37, C38, C39, C40, C43, C44, C45: 100nF, 0402C, symbol MCD_TOOLS:U_STM32Fx_1_Capacitor_ST_MCD_TOOLS.SchLib
- removed C41, C42: 2.2uF, TAN-A, symbol MCD_TOOLS:U_STM32Fx_3_Cap Low ESR_MCD_TOOLS.SchLib
- removed L1: BEAD, 0603L, symbol MCD_TOOLS:U_STM32Fx_1_Inductor_MCD_TOOLS.SchLib
- removed R52: 0, 0402R, symbol MCD_TOOLS:U_STM32Fx_1_Resistor_ST_MCD_TOOLS.SchLib
- removed R53, R54, R56, R58: 0, 0402R, symbol MCD_TOOLS:U_STM32Fx_0_Resistor_ST_MCD_TOOLS.SchLib
- removed R57: 220, 0402R, symbol MCD_TOOLS:U_STM32Fx_0_Resistor_ST_MCD_TOOLS.SchLib
- removed R59: [N/A], 0402R, symbol MCD_TOOLS:U_STM32Fx_0_Resistor_ST_MCD_TOOLS.SchLib
- removed R61: 510, 0402R, symbol MCD_TOOLS:U_STM32Fx_0_Resistor_ST_MCD_TOOLS.SchLib
- removed SB16, SB17, SB18, SB19, SB20, SB21, SB22, SB23, SB24, SB25: Circuit Breaker, JP2_SMD, symbol MB915:U_STM32Fx_0_Circuit Breaker_MB915.SCHLIB
- removed U5: STM32F429ZIT6, TQFP144, symbol MCD_TOOLS:U_STM32Fx_0_STM32F429ZIT6U_MCD_TOOLS.SchLib
- removed X2: MC306-G-06Q-32.768, MC306-CRYSTAL, symbol MCD_TOOLS:U_STM32Fx_2_mirrored_XTAL_32K_MCD_TOOLS.SchLib
- removed X3: 8MHz, XTAL1, symbol MCD_TOOLS:U_STM32Fx_1_XTAL_MCD_TOOLS.SchLib_0
- added C (x15): 100nF, 0402C, symbol MCD_TOOLS:root_1_Capacitor_ST_MCD_TOOLS.SchLib
- added C (x2): 20pF, 0402C, symbol MCD_TOOLS:root_0_Capacitor_ST_MCD_TOOLS.SchLib
- added C: 1uF, TAN-A, symbol Miscellaneous Devices:root_1_Cap Pol1_Miscellaneous Devices.IntLib
- added C (x2): 6.8pF, 0402C, symbol MCD_TOOLS:root_0_Capacitor_ST_MCD_TOOLS.SchLib
- added C: 1uF, 0603C, symbol MCD_TOOLS:root_0_Capacitor_ST_MCD_TOOLS.SchLib
- added C (x2): 2.2uF, TAN-A, symbol MCD_TOOLS:root_3_Cap Low ESR_MCD_TOOLS.SchLib
- added C: 1uF, TAN-A, symbol Miscellaneous Devices:root_3_Cap Pol1_Miscellaneous Devices.IntLib
- added L: BEAD, 0603L, symbol MCD_TOOLS:root_1_Inductor_MCD_TOOLS.SchLib
- added R: 510, 0402R, symbol MCD_TOOLS:root_0_Resistor_ST_MCD_TOOLS.SchLib
- added R (x4): 0, 0402R, symbol MCD_TOOLS:root_0_Resistor_ST_MCD_TOOLS.SchLib
- added R: [N/A], 0402R, symbol MCD_TOOLS:root_0_Resistor_ST_MCD_TOOLS.SchLib
- added R: 0, 0402R, symbol MCD_TOOLS:root_1_Resistor_ST_MCD_TOOLS.SchLib
- added R: 220, 0402R, symbol MCD_TOOLS:root_0_Resistor_ST_MCD_TOOLS.SchLib
- added SB (x10): Circuit Breaker, JP2_SMD, symbol MB915:root_0_Circuit Breaker_MB915.SCHLIB
- added U (x2): STM32F429ZIT6, TQFP144, symbol MCD_TOOLS:root_0_STM32F429ZIT6U_MCD_TOOLS.SchLib
- added X: 8MHz, XTAL1, symbol MCD_TOOLS:root_1_XTAL_MCD_TOOLS.SchLib_0
- added X: MC306-G-06Q-32.768, MC306-CRYSTAL, symbol MCD_TOOLS:root_2_mirrored_XTAL_32K_MCD_TOOLS.SchLib
Connections:
- net A0: now also U.10 (PF0)
- net A1: now also U.11 (PF1)
- net A10: now also U.56 (PG0)
- net A11: now also U.57 (PG1)
- net A2: now also U.12 (PF2)
- net A3: now also U.13 (PF3)
- net A4: now also U.14 (PF4)
- net A5: now also U.15 (PF5)
- net A6: now also U.50 (PF12)
- net A7: now also U.53 (PF13)
- net A8: now also U.54 (PF14)
- net A9: now also U.55 (PF15)
- net ACP_RST: now also U.43 (PA7)
- net B2: now also U.122 (PD6)
- net B3: now also U.126 (PG11)
- net B4: now also U.127 (PG12)
- net B5: now also U.37 (PA3)
- net B6: now also U.139 (PB8)
- net B7: now also U.140 (PB9)
- net BA0: now also U.89 (PG4)
- net BA1: now also U.90 (PG5)
- net BOOT0: now also R.2, R.2, U.138 (BOOT0)
- net CSX: now also U.28 (PC2)
- net D0: now also U.85 (PD14)
- net D1: now also U.86 (PD15)
- net D10: now also U.66 (PE13)
- net D11: now also U.67 (PE14)
- net D12: now also U.68 (PE15)
- net D13: now also U.77 (PD8)
- net D14: now also U.78 (PD9)
- net D15: now also U.79 (PD10)
- net D2: now also U.114 (PD0)
- net D3: now also U.115 (PD1)
- net D4: now also U.58 (PE7)
- net D5: now also U.59 (PE8)
- net D6: now also U.60 (PE9)
- net D7: now also U.63 (PE10)
- net D8: now also U.64 (PE11)
- net D9: now also U.65 (PE12)
- net DCX_SCL: now also U.19 (PF7)
- net DOTCLK: now also U.92 (PG7)
- net ENABLE: now also U.22 (PF10)
- net G2: now also U.42 (PA6)
- net G3: now also U.125 (PG10)
- net G4: now also U.69 (PB10)
- net G5: now also U.70 (PB11)
- net G6: now also U.97 (PC7)
- net G7: now also U.117 (PD3)
- net GND: now also C.1, C.1, C.1, C.1, C.1, C.1, C.1, C.1, C.1, C.1, C.1, C.1, C.1, C.1, C.1, C.2, C.2, C.2, C.2, C.2, C.2, C.2, C.2, C.2, SB.1, U.142 (PE1)
- net HSYNC: now also U.96 (PC6)
- net I2C3_SCL: now also U.100 (PA8)
- net I2C3_SDA: now also U.99 (PC9)
- net IM0: now also SB.2
- net IM1: now also SB.2
- net IM2: now also SB.2
- net IM3: now also SB.2
- net MCO: now also SB.1
- net MEMS_INT1: now also U.35 (PA1)
- net MEMS_INT2: now also U.36 (PA2)
- net NBL0: now also U.141 (PE0)
- net NBL1: now also U.142 (PE1)
- net NCS_MEMS_SPI: now also U.27 (PC1)
- net NRST: now also U.25 (NRST)
- net OTG_FS_DM: now also U.75 (PB14)
- net OTG_FS_DP: now also U.76 (PB15)
- net OTG_FS_ID: now also U.73 (PB12)
- net OTG_FS_OC: now also U.45 (PC5)
- net OTG_FS_PSO: now also U.44 (PC4)
- net PA0: now also U.34 (PA0-WKUP1)
- net PA10: now also U.102 (PA10)
- net PA11: now also U.103 (PA11)
- net PA12: now also U.104 (PA12)
- net PA13: now also U.105 (PA13)
- net PA14: now also U.109 (PA14)
- net PA5: now also U.41 (PA5)
- net PA9: now also U.101 (PA9)
- net PB0: now also U.46 (PB0)
- net PB1: now also U.47 (PB1)
- net PB2: now also U.48 (PB2/BOOT1)
- net PB3: now also U.133 (PB3)
- net PB4: now also U.134 (PB4)
- net PB7: now also U.137 (PB7)
- net PC10: now also U.111 (PC10)
- net PC11: now also U.112 (PC11)
- net PC12: now also U.113 (PC12)
- net PC13: now also U.7 (PC13-WKUP2)
- net PC14: now also SB.1
- net PC14-OSC32_IN: now also R.1, SB.2, U.8 (PC14-OSC32_IN)
- net PC15: now also SB.1
- net PC15-OSC32_OUT: now also R.1, SB.2, U.9 (PC15-OSC32_OUT)
- net PC3: now also U.29 (PC3)
- net PC8: now also U.98 (PC8)
- net PD2: now also SB.1, U.116 (PD2)
- net PD4: now also SB.1, U.118 (PD4)
- net PD5: now also SB.1, U.119 (PD5)
- net PD7: now also SB.1, U.123 (PD7)
- net PE2: now also U.1 (PE2)
- net PE3: now also U.2 (PE3)
- net PE4: now also U.3 (PE4)
- net PE5: now also U.4 (PE5)
- net PE6: now also U.5 (PE6)
- net PF6: now also U.18 (PF6)
- net PG13: now also U.128 (PG13)
- net PG14: now also U.129 (PG14)
- net PG2: now also U.87 (PG2)
- net PG3: now also U.88 (PG3)
- net PG6: now also U.91 (PG6)
- net PG9: now also U.124 (PG9)
- net PH0: now also SB.1
- net PH0-OSC_IN: now also R.1, SB.2, SB.2, U.23 (PH0-OSC_IN)
- net PH1: now also SB.1
- net PH1-OSC_OUT: now also R.1, SB.2, U.24 (PH1-OSC_OUT)
- net RDX: now also U.81 (PD12)
- net SDA: now also U.21 (PF9)
- net SDCKE1: now also U.135 (PB5)
- net SDCLK: now also U.93 (PG8)
- net SDNCAS: now also U.132 (PG15)
- net SDNE1: now also U.136 (PB6)
- net SDNRAS: now also U.49 (PF11)
- net SDNWE: now also U.26 (PC0)
- net SPI5_MISO: now also U.20 (PF8)
- net TE: now also U.80 (PD11)
- net TP_INT1: now also U.110 (PA15)
- net VBUS_FS: now also U.74 (PB13)
- net VDD: now also C.2, C.2, C.2, C.2, C.2, C.2, C.2, C.2, C.2, C.2, C.2, C.2, C.2, L.1, R.1, R.2, U.100 (PA8), U.101 (PA9), U.102 (PA10), U.103 (PA11), U.104 (PA12), U.105 (PA13), U.109 (PA14), U.110 (PA15), U.40 (PA4), U.41 (PA5), U.42 (PA6), U.43 (PA7)
- net VSYNC: now also U.40 (PA4)
- net WRX_DCX: now also U.82 (PD13)
- new net: C.1, R.2, X.2 (OSC2)
- new net: R.1, SB.2
- new net: C.1, R.2, X.1 (OSC1)
- new net: C.1, C.2, L.2, R.1, U.34 (PA0-WKUP1)
- new net: C.1, C.1, R.2, U.36 (PA2)
- new net: C.2, R.1, U.46 (PB0)
- new net: C.1, U.85 (PD14), U.86 (PD15)
- new net: C.1, R.2, X.1
- new net: C.1, R.2, X.4

Commit message: KILL ME!!!!!!!!!!!
Parts:
- removed C (x15): 100nF, 0402C, symbol MCD_TOOLS:root_1_Capacitor_ST_MCD_TOOLS.SchLib
- removed C (x2): 20pF, 0402C, symbol MCD_TOOLS:root_0_Capacitor_ST_MCD_TOOLS.SchLib
- removed C: 1uF, TAN-A, symbol Miscellaneous Devices:root_1_Cap Pol1_Miscellaneous Devices.IntLib
- removed C (x2): 6.8pF, 0402C, symbol MCD_TOOLS:root_0_Capacitor_ST_MCD_TOOLS.SchLib
- removed C: 1uF, 0603C, symbol MCD_TOOLS:root_0_Capacitor_ST_MCD_TOOLS.SchLib
- removed C (x2): 2.2uF, TAN-A, symbol MCD_TOOLS:root_3_Cap Low ESR_MCD_TOOLS.SchLib
- removed C: 1uF, TAN-A, symbol Miscellaneous Devices:root_3_Cap Pol1_Miscellaneous Devices.IntLib
- removed L: BEAD, 0603L, symbol MCD_TOOLS:root_1_Inductor_MCD_TOOLS.SchLib
- removed R: 510, 0402R, symbol MCD_TOOLS:root_0_Resistor_ST_MCD_TOOLS.SchLib
- removed R (x4): 0, 0402R, symbol MCD_TOOLS:root_0_Resistor_ST_MCD_TOOLS.SchLib
- removed R: [N/A], 0402R, symbol MCD_TOOLS:root_0_Resistor_ST_MCD_TOOLS.SchLib
- removed R: 0, 0402R, symbol MCD_TOOLS:root_1_Resistor_ST_MCD_TOOLS.SchLib
- removed R: 220, 0402R, symbol MCD_TOOLS:root_0_Resistor_ST_MCD_TOOLS.SchLib
- removed SB (x10): Circuit Breaker, JP2_SMD, symbol MB915:root_0_Circuit Breaker_MB915.SCHLIB
- removed U (x2): STM32F429ZIT6, TQFP144, symbol MCD_TOOLS:root_0_STM32F429ZIT6U_MCD_TOOLS.SchLib
- removed X: 8MHz, XTAL1, symbol MCD_TOOLS:root_1_XTAL_MCD_TOOLS.SchLib_0
- removed X: MC306-G-06Q-32.768, MC306-CRYSTAL, symbol MCD_TOOLS:root_2_mirrored_XTAL_32K_MCD_TOOLS.SchLib
- added C20, C21: 20pF, 0402C, symbol MCD_TOOLS:U_STM32Fx_0_Capacitor_ST_MCD_TOOLS.SchLib
- added C23, C24: 6.8pF, 0402C, symbol MCD_TOOLS:U_STM32Fx_0_Capacitor_ST_MCD_TOOLS.SchLib
- added C25: 1uF, TAN-A, symbol Miscellaneous Devices:U_STM32Fx_1_Cap Pol1_Miscellaneous Devices.IntLib
- added C26: 1uF, TAN-A, symbol Miscellaneous Devices:U_STM32Fx_3_Cap Pol1_Miscellaneous Devices.IntLib
- added C28: 1uF, 0603C, symbol MCD_TOOLS:U_STM32Fx_0_Capacitor_ST_MCD_TOOLS.SchLib
- added C29, C30, C31, C32, C33, C34, C35, C36, C37, C38, C39, C40, C43, C44, C45: 100nF, 0402C, symbol MCD_TOOLS:U_STM32Fx_1_Capacitor_ST_MCD_TOOLS.SchLib
- added C41, C42: 2.2uF, TAN-A, symbol MCD_TOOLS:U_STM32Fx_3_Cap Low ESR_MCD_TOOLS.SchLib
- added L1: BEAD, 0603L, symbol MCD_TOOLS:U_STM32Fx_1_Inductor_MCD_TOOLS.SchLib
- added R52: 0, 0402R, symbol MCD_TOOLS:U_STM32Fx_1_Resistor_ST_MCD_TOOLS.SchLib
- added R53, R54, R56, R58: 0, 0402R, symbol MCD_TOOLS:U_STM32Fx_0_Resistor_ST_MCD_TOOLS.SchLib
- added R57: 220, 0402R, symbol MCD_TOOLS:U_STM32Fx_0_Resistor_ST_MCD_TOOLS.SchLib
- added R59: [N/A], 0402R, symbol MCD_TOOLS:U_STM32Fx_0_Resistor_ST_MCD_TOOLS.SchLib
- added R61: 510, 0402R, symbol MCD_TOOLS:U_STM32Fx_0_Resistor_ST_MCD_TOOLS.SchLib
- added SB16, SB17, SB18, SB19, SB20, SB21, SB22, SB23, SB24, SB25: Circuit Breaker, JP2_SMD, symbol MB915:U_STM32Fx_0_Circuit Breaker_MB915.SCHLIB
- added U5: STM32F429ZIT6, TQFP144, symbol MCD_TOOLS:U_STM32Fx_0_STM32F429ZIT6U_MCD_TOOLS.SchLib
- added X2: MC306-G-06Q-32.768, MC306-CRYSTAL, symbol MCD_TOOLS:U_STM32Fx_2_mirrored_XTAL_32K_MCD_TOOLS.SchLib
- added X3: 8MHz, XTAL1, symbol MCD_TOOLS:U_STM32Fx_1_XTAL_MCD_TOOLS.SchLib_0
Connections:
- net A0: now also U5.10 (PF0)
- net A1: now also U5.11 (PF1)
- net A10: now also U5.56 (PG0)
- net A11: now also U5.57 (PG1)
- net A2: now also U5.12 (PF2)
- net A3: now also U5.13 (PF3)
- net A4: now also U5.14 (PF4)
- net A5: now also U5.15 (PF5)
- net A6: now also U5.50 (PF12)
- net A7: now also U5.53 (PF13)
- net A8: now also U5.54 (PF14)
- net A9: now also U5.55 (PF15)
- net ACP_RST: now also U5.43 (PA7)
- net B2: now also U5.122 (PD6)
- net B3: now also U5.126 (PG11)
- net B4: now also U5.127 (PG12)
- net B5: now also U5.37 (PA3)
- net B6: now also U5.139 (PB8)
- net B7: now also U5.140 (PB9)
- net BA0: now also U5.89 (PG4)
- net BA1: now also U5.90 (PG5)
- net BOOT0: now also R59.2, R61.2, U5.138 (BOOT0)
- net CSX: now also U5.28 (PC2)
- net D0: now also U5.85 (PD14)
- net D1: now also U5.86 (PD15)
- net D10: now also U5.66 (PE13)
- net D11: now also U5.67 (PE14)
- net D12: now also U5.68 (PE15)
- net D13: now also U5.77 (PD8)
- net D14: now also U5.78 (PD9)
- net D15: now also U5.79 (PD10)
- net D2: now also U5.114 (PD0)
- net D3: now also U5.115 (PD1)
- net D4: now also U5.58 (PE7)
- net D5: now also U5.59 (PE8)
- net D6: now also U5.60 (PE9)
- net D7: now also U5.63 (PE10)
- net D8: now also U5.64 (PE11)
- net D9: now also U5.65 (PE12)
- net DCX_SCL: now also U5.19 (PF7)
- net DOTCLK: now also U5.92 (PG7)
- net ENABLE: now also U5.22 (PF10)
- net G2: now also U5.42 (PA6)
- net G3: now also U5.125 (PG10)
- net G4: now also U5.69 (PB10)
- net G5: now also U5.70 (PB11)
- net G6: now also U5.97 (PC7)
- net G7: now also U5.117 (PD3)
- net GND: now also C20.2, C21.2, C23.2, C24.2, C25.2, C26.2, C28.1, C29.1, C30.2, C31.1, C32.1, C33.1, C34.1, C35.1, C36.1, C37.1, C38.1, C39.1, C40.1, C41.2, C42.2, C43.1, C44.1, C45.1, SB21.1, U5.107 (VSS_2), U5.120 (VSS_10), U5.130 (VSS_11), U5.16 (VSS_5), U5.31 (VSSA), U5.38 (VSS_4), U5.51 (VSS_6), U5.61 (VSS_7), U5.83 (VSS_8), U5.94 (VSS_9)
- net HSYNC: now also U5.96 (PC6)
- net I2C3_SCL: now also U5.100 (PA8)
- net I2C3_SDA: now also U5.99 (PC9)
- net IM0: now also SB25.2
- net IM1: now also SB24.2
- net IM2: now also SB23.2
- net IM3: now also SB22.2
- net MCO: now also SB18.1
- net MEMS_INT1: now also U5.35 (PA1)
- net MEMS_INT2: now also U5.36 (PA2)
- net NBL0: now also U5.141 (PE0)
- net NBL1: now also U5.142 (PE1)
- net NCS_MEMS_SPI: now also U5.27 (PC1)
- net NRST: now also U5.25 (NRST)
- net OTG_FS_DM: now also U5.75 (PB14)
- net OTG_FS_DP: now also U5.76 (PB15)
- net OTG_FS_ID: now also U5.73 (PB12)
- net OTG_FS_OC: now also U5.45 (PC5)
- net OTG_FS_PSO: now also U5.44 (PC4)
- net PA0: now also U5.34 (PA0-WKUP1)
- net PA10: now also U5.102 (PA10)
- net PA11: now also U5.103 (PA11)
- net PA12: now also U5.104 (PA12)
- net PA13: now also U5.105 (PA13)
- net PA14: now also U5.109 (PA14)
- net PA5: now also U5.41 (PA5)
- net PA9: now also U5.101 (PA9)
- net PB0: now also U5.46 (PB0)
- net PB1: now also U5.47 (PB1)
- net PB2: now also U5.48 (PB2/BOOT1)
- net PB3: now also U5.133 (PB3)
- net PB4: now also U5.134 (PB4)
- net PB7: now also U5.137 (PB7)
- net PC10: now also U5.111 (PC10)
- net PC11: now also U5.112 (PC11)
- net PC12: now also U5.113 (PC12)
- net PC13: now also U5.7 (PC13-WKUP2)
- net PC14: now also SB16.1
- net PC14-OSC32_IN: now also R53.1, SB16.2, U5.8 (PC14-OSC32_IN)
- net PC15: now also SB17.1
- net PC15-OSC32_OUT: now also R54.1, SB17.2, U5.9 (PC15-OSC32_OUT)
- net PC3: now also U5.29 (PC3)
- net PC8: now also U5.98 (PC8)
- net PD2: now also SB25.1, U5.116 (PD2)
- net PD4: now also SB24.1, U5.118 (PD4)
- net PD5: now also SB23.1, U5.119 (PD5)
- net PD7: now also SB22.1, U5.123 (PD7)
- net PE2: now also U5.1 (PE2)
- net PE3: now also U5.2 (PE3)
- net PE4: now also U5.3 (PE4)
- net PE5: now also U5.4 (PE5)
- net PE6: now also U5.5 (PE6)
- net PF6: now also U5.18 (PF6)
- net PG13: now also U5.128 (PG13)
- net PG14: now also U5.129 (PG14)
- net PG2: now also U5.87 (PG2)
- net PG3: now also U5.88 (PG3)
- net PG6: now also U5.91 (PG6)
- net PG9: now also U5.124 (PG9)
- net PH0: now also SB19.1
- net PH0-OSC_IN: now also R56.1, SB18.2, SB19.2, U5.23 (PH0-OSC_IN)
- net PH1: now also SB20.1
- net PH1-OSC_OUT: now also R57.1, SB20.2, U5.24 (PH1-OSC_OUT)
- net RDX: now also U5.81 (PD12)
- net SDA: now also U5.21 (PF9)
- net SDCKE1: now also U5.135 (PB5)
- net SDCLK: now also U5.93 (PG8)
- net SDNCAS: now also U5.132 (PG15)
- net SDNE1: now also U5.136 (PB6)
- net SDNRAS: now also U5.49 (PF11)
- net SDNWE: now also U5.26 (PC0)
- net SPI5_MISO: now also U5.20 (PF8)
- net TE: now also U5.80 (PD11)
- net TP_INT1: now also U5.110 (PA15)
- net VBUS_FS: now also U5.74 (PB13)
- net VDD: now also C29.2, C32.2, C33.2, C34.2, C35.2, C36.2, C37.2, C38.2, C39.2, C40.2, C43.2, C44.2, C45.2, L1.1, R52.2, R59.1, U5.108 (VDD_2), U5.121 (VDD_10), U5.131 (VDD_11), U5.143 (PDR_ON), U5.144 (VDD_3), U5.17 (VDD_5), U5.30 (VDD_12), U5.39 (VDD_4), U5.52 (VDD_6), U5.62 (VDD_7), U5.72 (VDD_1), U5.84 (VDD_8), U5.95 (VDD_9)
- net VSYNC: now also U5.40 (PA4)
- net WRX_DCX: now also U5.82 (PD13)
- new net: C20.1, R56.2, X3.2 (OSC2)
- new net: C42.1, U5.106 (VCAP2)
- new net: C25.1, C30.1, R58.2, U5.32 (VREF+)
- new net: C26.1, C31.2, L1.2, R58.1, U5.33 (VDDA)
- new net: C28.2, R52.1, U5.6 (VBAT)
- new net: C41.1, U5.71 (VCAP1)
- new net: R61.1, SB21.2
- new net: C21.1, R57.2, X3.1 (OSC1)
- new net: C24.1, R54.2, X2.1
- new net: C23.1, R53.2, X2.4
