File: docs/mb1075_bdp/MB1075E/Altium_Designer/ST_LINK_V2.kicad_sch (KiCad schematic)
At the start: 68 parts, among them CN1 USB-MINI-typeB, CN2 Header 6, CN4 Header 4, U1 LD3985M33R, U2 STM32F103CBT6, X1 8MHz

Commit message: save before i break everything out instead idk why i didnt do that
Parts:
- removed C1, C27, C4, C46, C47, C6, C9: 100nF, 0402C, symbol MCD_TOOLS:U_ST_LINK_1_Capacitor_ST_MCD_TOOLS.SchLib
- removed C16, C17, C18: 20pF, 0402C, symbol MCD_TOOLS:U_ST_LINK_1_Capacitor_ST_MCD_TOOLS.SchLib
- removed C2: 1µF_X5R_0603, 0603C, symbol MB963_1:U_ST_LINK_1_CAP SMD 0603 X5R 1µF 25V 10%_MB963_1.SCHLIB
- removed C3: 10nF_X7R_0603, 0603C, symbol MB963_1:U_ST_LINK_1_CAP SMD 0603 X7R 10000PF 50V 10%_MB963_1.SCHLIB
- removed C5: 1µF_X5R_0603, 0603C, symbol MB963_1:U_ST_LINK_3_CAP SMD 0603 X5R 1µF 25V 10%_MB963_1.SCHLIB
- removed CN1: USB-MINI-typeB, USB-MINI-B-SMD, symbol MCD_TOOLS:U_ST_LINK_0_USB-MINI-typeB connector_MCD_TOOLS.SchLib_0
- removed CN2: Header 6, HDR1X6, symbol Miscellaneous Connectors:U_ST_LINK_0_mirrored_Header 6_Miscellaneous Connectors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
- removed CN4: Header 4, Header 4, symbol MB963_1:U_ST_LINK_3_mirrored_Header 4_MB963_1.SCHLIB
- removed D1, D2, D3: BAT60JFILM, SOD323/A, symbol MCD_TOOLS:U_ST_LINK_0_BAT60JFILM_MCD_TOOLS.SchLib
- removed HW1, HW2, HW3, HW4, HW5: Shunt Black 2.54mm, symbol MB1075:U_ST_LINK_0_Shunt Black 2.54mm_MB1075.SCHLIB
- removed JP1, JP2, JP3: (no value), SIP2/2.54, symbol *:U_ST_LINK_0_JP2_*
- removed JP4: JP2, SIP2/2.54, symbol MCD_TOOLS:U_ST_LINK_1_JP2_MCD_TOOLS.SchLib
- removed LD1: LD_BICOLOR_CMS, HSMF-A201, symbol MCD_TOOLS:U_ST_LINK_0_mirrored_LD_BICOLOR_CMS_MCD_TOOLS.SchLib
- removed LD2: LED, red, 0603D, symbol MCD_TOOLS:U_ST_LINK_0_LED_red_MCD_TOOLS.SchLib_0
- removed R1, R2, R28: 100, 0402R, symbol MCD_TOOLS:U_ST_LINK_0_Resistor_ST_MCD_TOOLS.SchLib
- removed R10: 1K5, 0402R, symbol MCD_TOOLS:U_ST_LINK_0_Resistor_ST_MCD_TOOLS.SchLib
- removed R11, R12, R3: 0, 0402R, symbol MCD_TOOLS:U_ST_LINK_0_Resistor_ST_MCD_TOOLS.SchLib
- removed R13: [NA], 0402R, symbol MCD_TOOLS:U_ST_LINK_0_Resistor_ST_MCD_TOOLS.SchLib
- removed R14, R15, R17, R20: 22, 0402R, symbol MCD_TOOLS:U_ST_LINK_0_Resistor_ST_MCD_TOOLS.SchLib
- removed R16: 100, 0402R, symbol MCD_TOOLS:U_ST_LINK_1_Resistor_ST_MCD_TOOLS.SchLib
- removed R18, R19: 4K7, 0402R, symbol MCD_TOOLS:U_ST_LINK_0_Resistor_ST_MCD_TOOLS.SchLib
- removed R21: 100K, 0402R, symbol MCD_TOOLS:U_ST_LINK_1_Resistor_ST_MCD_TOOLS.SchLib
- removed R4: 1K, 0402R, symbol MCD_TOOLS:U_ST_LINK_1_Resistor_ST_MCD_TOOLS.SchLib
- removed R5: 10K, 0402R, symbol MCD_TOOLS:U_ST_LINK_1_Resistor_ST_MCD_TOOLS.SchLib
- removed R6, R7: 10K, 0402R, symbol MCD_TOOLS:U_ST_LINK_0_Resistor_ST_MCD_TOOLS.SchLib
- removed R8, R9: 100K, 0402R, symbol MCD_TOOLS:U_ST_LINK_0_Resistor_ST_MCD_TOOLS.SchLib
- removed SB10: Circuit Breaker, JP2_SMD, symbol MB915:U_ST_LINK_1_Circuit Breaker_MB915.SCHLIB
- removed SB11, SB15, SB9: Circuit Breaker, JP2_SMD, symbol MCD_TOOLS:U_ST_LINK_0_Circuit Breaker_MCD_TOOLS.SCHLIB
- removed SB12, SB13, SB14, SB3, SB4, SB5, SB6, SB7, SB8: Circuit Breaker, JP2_SMD, symbol MB915:U_ST_LINK_0_Circuit Breaker_MB915.SCHLIB
- removed U1: LD3985M33R, SOT-23-5L, symbol MCD_TOOLS:U_ST_LINK_0_LD3985M33R_MCD_TOOLS.SchLib
- removed U2: STM32F103CBT6, QFP48 7x7, symbol MCD_TOOLS:U_ST_LINK_0_STM32F103CBT6_MCD_TOOLS.SchLib
- removed X1: 8MHz, XTAL1, symbol MCD_TOOLS:U_ST_LINK_0_XTAL_MCD_TOOLS.SchLib_0
- added C (x7): 100nF, 0402C, symbol MCD_TOOLS:root_1_Capacitor_ST_MCD_TOOLS.SchLib
- added C (x3): 20pF, 0402C, symbol MCD_TOOLS:root_1_Capacitor_ST_MCD_TOOLS.SchLib
- added C: 10nF_X7R_0603, 0603C, symbol MB963_1:root_1_CAP SMD 0603 X7R 10000PF 50V 10%_MB963_1.SCHLIB
- added C: 1µF_X5R_0603, 0603C, symbol MB963_1:root_3_CAP SMD 0603 X5R 1µF 25V 10%_MB963_1.SCHLIB
- added C: 1µF_X5R_0603, 0603C, symbol MB963_1:root_1_CAP SMD 0603 X5R 1µF 25V 10%_MB963_1.SCHLIB
- added CN: Header 4, Header 4, symbol MB963_1:root_3_mirrored_Header 4_MB963_1.SCHLIB
- added CN: Header 6, HDR1X6, symbol Miscellaneous Connectors:root_0_mirrored_Header 6_Miscellaneous Connectors.IntL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
- added CN: USB-MINI-typeB, USB-MINI-B-SMD, symbol MCD_TOOLS:root_0_USB-MINI-typeB connector_MCD_TOOLS.SchLib_0
- added D (x3): BAT60JFILM, SOD323/A, symbol MCD_TOOLS:root_0_BAT60JFILM_MCD_TOOLS.SchLib
- added HW (x5): Shunt Black 2.54mm, symbol MB1075:root_0_Shunt Black 2.54mm_MB1075.SCHLIB
- added JP: JP2, SIP2/2.54, symbol MCD_TOOLS:root_1_JP2_MCD_TOOLS.SchLib
- added JP (x3): (no value), SIP2/2.54, symbol *:root_0_JP2_*
- added LD: LED, red, 0603D, symbol MCD_TOOLS:root_0_LED_red_MCD_TOOLS.SchLib_0
- added LD: LD_BICOLOR_CMS, HSMF-A201, symbol MCD_TOOLS:root_0_mirrored_LD_BICOLOR_CMS_MCD_TOOLS.SchLib
- added R: 10K, 0402R, symbol MCD_TOOLS:root_1_Resistor_ST_MCD_TOOLS.SchLib
- added R (x2): 10K, 0402R, symbol MCD_TOOLS:root_0_Resistor_ST_MCD_TOOLS.SchLib
- added R: 100, 0402R, symbol MCD_TOOLS:root_1_Resistor_ST_MCD_TOOLS.SchLib
- added R (x3): 100, 0402R, symbol MCD_TOOLS:root_0_Resistor_ST_MCD_TOOLS.SchLib
- added R (x4): 22, 0402R, symbol MCD_TOOLS:root_0_Resistor_ST_MCD_TOOLS.SchLib
- added R (x2): 100K, 0402R, symbol MCD_TOOLS:root_0_Resistor_ST_MCD_TOOLS.SchLib
- added R (x3): 0, 0402R, symbol MCD_TOOLS:root_0_Resistor_ST_MCD_TOOLS.SchLib
- added R: 1K5, 0402R, symbol MCD_TOOLS:root_0_Resistor_ST_MCD_TOOLS.SchLib
- added R (x2): 4K7, 0402R, symbol MCD_TOOLS:root_0_Resistor_ST_MCD_TOOLS.SchLib
- added R: 1K, 0402R, symbol MCD_TOOLS:root_1_Resistor_ST_MCD_TOOLS.SchLib
- added R: 100K, 0402R, symbol MCD_TOOLS:root_1_Resistor_ST_MCD_TOOLS.SchLib
- added R: [NA], 0402R, symbol MCD_TOOLS:root_0_Resistor_ST_MCD_TOOLS.SchLib
- added SB (x9): Circuit Breaker, JP2_SMD, symbol MB915:root_0_Circuit Breaker_MB915.SCHLIB
- added SB (x3): Circuit Breaker, JP2_SMD, symbol MCD_TOOLS:root_0_Circuit Breaker_MCD_TOOLS.SCHLIB
- added SB: Circuit Breaker, JP2_SMD, symbol MB915:root_1_Circuit Breaker_MB915.SCHLIB
- added U: STM32F103CBT6, QFP48 7x7, symbol MCD_TOOLS:root_0_STM32F103CBT6_MCD_TOOLS.SchLib
- added U: LD3985M33R, SOT-23-5L, symbol MCD_TOOLS:root_0_LD3985M33R_MCD_TOOLS.SchLib
- added X: 8MHz, XTAL1, symbol MCD_TOOLS:root_0_XTAL_MCD_TOOLS.SchLib_0
Connections:
- net 3V: now also C.2, C.2, C.2, C.2, D.2 (K), JP.1 (COMMON), R.1, R.2, R.2, R.2, R.2, SB.2, U.1 (VBAT), U.24 (VDD_1), U.36 (VDD_2), U.48 (VDD_3), U.9 (VDDA)
- net 5V: now also C.2, C.2, D.2 (K), U.1 (Vin), U.3 (CE)
- net AIN_1: now also R.2, R.2, R.2, U.10 (PA0)
- net GND: now also C.1, C.1, C.1, C.1, C.1, C.1, C.1, C.1, C.1, C.1, C.2, C.2, C.2, CN.3, CN.5 (GND), CN.6 (SHELL), JP.1 (COMMON), JP.1 (COMMON), JP.2 (NO), JP.2 (NO), LD.1, LD.2, R.1, R.1, R.1, R.1, R.2, R.2, SB.1, SB.2, U.2 (GND), U.20 (PB2/BOOT1), U.23 (VSS_1), U.35 (VSS_2), U.47 (VSS_3), U.8 (VSSA)
- net LED_STLINK: now also R.1, R.1, U.30 (PA9)
- net MCO: now also C.2, R.2
- net NRST: now also SB.2
- net OSC_IN: now also C.1, U.5 (OSCIN), X.2 (OSC2)
- net OSC_OUT: now also C.1, U.6 (OSCOUT), X.1 (OSC1)
- net PA10: now also SB.1
- net PA13: now also SB.1
- net PA14: now also SB.1
- net PA9: now also SB.1
- net PB3: now also SB.2
- net STLINK_RX: now also JP.1 (COMMON), SB.2, U.13 (PA3)
- net STLINK_TX: now also JP.2 (NO), SB.2, U.12 (PA2)
- net STM_JTCK: now also SB.2, U.37 (JTCK/SWCLK)
- net STM_JTMS: now also SB.2, U.34 (JTMS/SWDIO)
- net STM_RST: now also C.2, R.1, SB.2, U.7 (NRST)
- net SWIM: now also U.22 (PB11), U.45 (PB8)
- net SWIM_IN: now also U.21 (PB10), U.43 (PB7), U.46 (PB9)
- net SWIM_RST: now also U.42 (PB6)
- net SWIM_RST_IN: now also U.41 (PB5)
- net T_JTCK: now also R.2, SB.1, U.15 (PA5), U.26 (PB13)
- net T_JTDI: now also U.17 (PA7)
- net T_JTDO: now also U.16 (PA6)
- net T_JTMS: now also R.2, R.2, SB.1, U.27 (PB14)
- net T_NRST: now also R.2, SB.1, U.18 (PB0)
- net T_SWDIO_IN: now also R.1, U.25 (PB12)
- net T_SWO: now also R.2, SB.1, U.31 (PA10)
- net U5V: now also CN.1 (VCC), D.1 (A)
- net USB_DM: now also R.2, U.32 (PA11)
- net USB_DP: now also R.2, U.33 (PA12)
- net VDD: now also JP.2 (NO)
- new net: CN.2, SB.1, SB.2
- new net: LD.1, R.1
- new net: CN.1, D.1 (A), R.1
- new net: R.2, U.2 (PC13)
- new net: CN.1, SB.1, SB.2
- new net: CN.3, SB.1, SB.2
- new net: CN.4, SB.1, SB.2
- new net: D.2 (K), R.1
- new net: R.1, U.29 (PA8)
- new net: LD.3, R.2
- new net: CN.5, R.1
- new net: CN.6, R.1
- new net: CN.2, R.1
- new net: CN.4, R.1
- new net: CN.4 (ID), R.1
- new net: C.1, C.2, D.1 (A), U.5 (Vout)
- new net: CN.2 (D-), R.1
- new net: CN.3 (D+), R.1, R.1
- new net: R.2, U.3 (PC14)
- new net: R.2, U.44 (BOOT0)
- new net: C.2, U.4 (BYPASS)
- new net: LD.4, R.1
- new net: LD.2, R.2

Commit message: KILL ME!!!!!!!!!!!
Parts:
- removed C (x7): 100nF, 0402C, symbol MCD_TOOLS:root_1_Capacitor_ST_MCD_TOOLS.SchLib
- removed C (x3): 20pF, 0402C, symbol MCD_TOOLS:root_1_Capacitor_ST_MCD_TOOLS.SchLib
- removed C: 10nF_X7R_0603, 0603C, symbol MB963_1:root_1_CAP SMD 0603 X7R 10000PF 50V 10%_MB963_1.SCHLIB
- removed C: 1µF_X5R_0603, 0603C, symbol MB963_1:root_3_CAP SMD 0603 X5R 1µF 25V 10%_MB963_1.SCHLIB
- removed C: 1µF_X5R_0603, 0603C, symbol MB963_1:root_1_CAP SMD 0603 X5R 1µF 25V 10%_MB963_1.SCHLIB
- removed CN: Header 4, Header 4, symbol MB963_1:root_3_mirrored_Header 4_MB963_1.SCHLIB
- removed CN: Header 6, HDR1X6, symbol Miscellaneous Connectors:root_0_mirrored_Header 6_Miscellaneous Connectors.IntL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
- removed CN: USB-MINI-typeB, USB-MINI-B-SMD, symbol MCD_TOOLS:root_0_USB-MINI-typeB connector_MCD_TOOLS.SchLib_0
- removed D (x3): BAT60JFILM, SOD323/A, symbol MCD_TOOLS:root_0_BAT60JFILM_MCD_TOOLS.SchLib
- removed HW (x5): Shunt Black 2.54mm, symbol MB1075:root_0_Shunt Black 2.54mm_MB1075.SCHLIB
- removed JP: JP2, SIP2/2.54, symbol MCD_TOOLS:root_1_JP2_MCD_TOOLS.SchLib
- removed JP (x3): (no value), SIP2/2.54, symbol *:root_0_JP2_*
- removed LD: LED, red, 0603D, symbol MCD_TOOLS:root_0_LED_red_MCD_TOOLS.SchLib_0
- removed LD: LD_BICOLOR_CMS, HSMF-A201, symbol MCD_TOOLS:root_0_mirrored_LD_BICOLOR_CMS_MCD_TOOLS.SchLib
- removed R: 10K, 0402R, symbol MCD_TOOLS:root_1_Resistor_ST_MCD_TOOLS.SchLib
- removed R (x2): 10K, 0402R, symbol MCD_TOOLS:root_0_Resistor_ST_MCD_TOOLS.SchLib
- removed R: 100, 0402R, symbol MCD_TOOLS:root_1_Resistor_ST_MCD_TOOLS.SchLib
- removed R (x3): 100, 0402R, symbol MCD_TOOLS:root_0_Resistor_ST_MCD_TOOLS.SchLib
- removed R (x4): 22, 0402R, symbol MCD_TOOLS:root_0_Resistor_ST_MCD_TOOLS.SchLib
- removed R (x2): 100K, 0402R, symbol MCD_TOOLS:root_0_Resistor_ST_MCD_TOOLS.SchLib
- removed R (x3): 0, 0402R, symbol MCD_TOOLS:root_0_Resistor_ST_MCD_TOOLS.SchLib
- removed R: 1K5, 0402R, symbol MCD_TOOLS:root_0_Resistor_ST_MCD_TOOLS.SchLib
- removed R (x2): 4K7, 0402R, symbol MCD_TOOLS:root_0_Resistor_ST_MCD_TOOLS.SchLib
- removed R: 1K, 0402R, symbol MCD_TOOLS:root_1_Resistor_ST_MCD_TOOLS.SchLib
- removed R: 100K, 0402R, symbol MCD_TOOLS:root_1_Resistor_ST_MCD_TOOLS.SchLib
- removed R: [NA], 0402R, symbol MCD_TOOLS:root_0_Resistor_ST_MCD_TOOLS.SchLib
- removed SB (x9): Circuit Breaker, JP2_SMD, symbol MB915:root_0_Circuit Breaker_MB915.SCHLIB
- removed SB (x3): Circuit Breaker, JP2_SMD, symbol MCD_TOOLS:root_0_Circuit Breaker_MCD_TOOLS.SCHLIB
- removed SB: Circuit Breaker, JP2_SMD, symbol MB915:root_1_Circuit Breaker_MB915.SCHLIB
- removed U: STM32F103CBT6, QFP48 7x7, symbol MCD_TOOLS:root_0_STM32F103CBT6_MCD_TOOLS.SchLib
- removed U: LD3985M33R, SOT-23-5L, symbol MCD_TOOLS:root_0_LD3985M33R_MCD_TOOLS.SchLib
- removed X: 8MHz, XTAL1, symbol MCD_TOOLS:root_0_XTAL_MCD_TOOLS.SchLib_0
- added C1, C27, C4, C46, C47, C6, C9: 100nF, 0402C, symbol MCD_TOOLS:U_ST_LINK_1_Capacitor_ST_MCD_TOOLS.SchLib
- added C16, C17, C18: 20pF, 0402C, symbol MCD_TOOLS:U_ST_LINK_1_Capacitor_ST_MCD_TOOLS.SchLib
- added C2: 1µF_X5R_0603, 0603C, symbol MB963_1:U_ST_LINK_1_CAP SMD 0603 X5R 1µF 25V 10%_MB963_1.SCHLIB
- added C3: 10nF_X7R_0603, 0603C, symbol MB963_1:U_ST_LINK_1_CAP SMD 0603 X7R 10000PF 50V 10%_MB963_1.SCHLIB
- added C5: 1µF_X5R_0603, 0603C, symbol MB963_1:U_ST_LINK_3_CAP SMD 0603 X5R 1µF 25V 10%_MB963_1.SCHLIB
- added CN1: USB-MINI-typeB, USB-MINI-B-SMD, symbol MCD_TOOLS:U_ST_LINK_0_USB-MINI-typeB connector_MCD_TOOLS.SchLib_0
- added CN2: Header 6, HDR1X6, symbol Miscellaneous Connectors:U_ST_LINK_0_mirrored_Header 6_Miscellaneous Connectors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
- added CN4: Header 4, Header 4, symbol MB963_1:U_ST_LINK_3_mirrored_Header 4_MB963_1.SCHLIB
- added D1, D2, D3: BAT60JFILM, SOD323/A, symbol MCD_TOOLS:U_ST_LINK_0_BAT60JFILM_MCD_TOOLS.SchLib
- added HW1, HW2, HW3, HW4, HW5: Shunt Black 2.54mm, symbol MB1075:U_ST_LINK_0_Shunt Black 2.54mm_MB1075.SCHLIB
- added JP1, JP2, JP3: (no value), SIP2/2.54, symbol *:U_ST_LINK_0_JP2_*
- added JP4: JP2, SIP2/2.54, symbol MCD_TOOLS:U_ST_LINK_1_JP2_MCD_TOOLS.SchLib
- added LD1: LD_BICOLOR_CMS, HSMF-A201, symbol MCD_TOOLS:U_ST_LINK_0_mirrored_LD_BICOLOR_CMS_MCD_TOOLS.SchLib
- added LD2: LED, red, 0603D, symbol MCD_TOOLS:U_ST_LINK_0_LED_red_MCD_TOOLS.SchLib_0
- added R1, R2, R28: 100, 0402R, symbol MCD_TOOLS:U_ST_LINK_0_Resistor_ST_MCD_TOOLS.SchLib
- added R10: 1K5, 0402R, symbol MCD_TOOLS:U_ST_LINK_0_Resistor_ST_MCD_TOOLS.SchLib
- added R11, R12, R3: 0, 0402R, symbol MCD_TOOLS:U_ST_LINK_0_Resistor_ST_MCD_TOOLS.SchLib
- added R13: [NA], 0402R, symbol MCD_TOOLS:U_ST_LINK_0_Resistor_ST_MCD_TOOLS.SchLib
- added R14, R15, R17, R20: 22, 0402R, symbol MCD_TOOLS:U_ST_LINK_0_Resistor_ST_MCD_TOOLS.SchLib
- added R16: 100, 0402R, symbol MCD_TOOLS:U_ST_LINK_1_Resistor_ST_MCD_TOOLS.SchLib
- added R18, R19: 4K7, 0402R, symbol MCD_TOOLS:U_ST_LINK_0_Resistor_ST_MCD_TOOLS.SchLib
- added R21: 100K, 0402R, symbol MCD_TOOLS:U_ST_LINK_1_Resistor_ST_MCD_TOOLS.SchLib
- added R4: 1K, 0402R, symbol MCD_TOOLS:U_ST_LINK_1_Resistor_ST_MCD_TOOLS.SchLib
- added R5: 10K, 0402R, symbol MCD_TOOLS:U_ST_LINK_1_Resistor_ST_MCD_TOOLS.SchLib
- added R6, R7: 10K, 0402R, symbol MCD_TOOLS:U_ST_LINK_0_Resistor_ST_MCD_TOOLS.SchLib
- added R8, R9: 100K, 0402R, symbol MCD_TOOLS:U_ST_LINK_0_Resistor_ST_MCD_TOOLS.SchLib
- added SB10: Circuit Breaker, JP2_SMD, symbol MB915:U_ST_LINK_1_Circuit Breaker_MB915.SCHLIB
- added SB11, SB15, SB9: Circuit Breaker, JP2_SMD, symbol MCD_TOOLS:U_ST_LINK_0_Circuit Breaker_MCD_TOOLS.SCHLIB
- added SB12, SB13, SB14, SB3, SB4, SB5, SB6, SB7, SB8: Circuit Breaker, JP2_SMD, symbol MB915:U_ST_LINK_0_Circuit Breaker_MB915.SCHLIB
- added U1: LD3985M33R, SOT-23-5L, symbol MCD_TOOLS:U_ST_LINK_0_LD3985M33R_MCD_TOOLS.SchLib
- added U2: STM32F103CBT6, QFP48 7x7, symbol MCD_TOOLS:U_ST_LINK_0_STM32F103CBT6_MCD_TOOLS.SchLib
- added X1: 8MHz, XTAL1, symbol MCD_TOOLS:U_ST_LINK_0_XTAL_MCD_TOOLS.SchLib_0
Connections:
- net 3V: now also C27.2, C4.2, C46.2, C47.2, D3.2 (K), JP3.1 (COMMON), R10.2, R18.1, R21.2, R3.2, R4.2, SB3.2, U2.1 (VBAT), U2.24 (VDD_1), U2.36 (VDD_2), U2.48 (VDD_3), U2.9 (VDDA)
- net 5V: now also C1.2, C2.2, D2.2 (K), U1.1 (Vin), U1.3 (CE)
- net AIN_1: now also R13.2, R18.2, R19.2, U2.10 (PA0)
- net GND: now also C1.1, C16.2, C17.2, C18.1, C2.1, C27.1, C3.1, C4.1, C46.1, C47.1, C5.2, C6.1, C9.1, CN1.5 (GND), CN1.6 (SHELL), CN2.3, JP1.1 (COMMON), JP1.2 (NO), JP2.1 (COMMON), JP2.2 (NO), LD1.1, LD2.2, R19.1, R5.2, R6.1, R7.1, R8.1, R9.2, SB10.1, SB7.2, U1.2 (GND), U2.20 (PB2/BOOT1), U2.23 (VSS_1), U2.35 (VSS_2), U2.47 (VSS_3), U2.8 (VSSA)
- net LED_STLINK: now also R1.1, R2.1, U2.30 (PA9)
- net MCO: now also C18.2, R28.2
- net NRST: now also SB12.2
- net OSC_IN: now also C16.1, U2.5 (OSCIN), X1.2 (OSC2)
- net OSC_OUT: now also C17.1, U2.6 (OSCOUT), X1.1 (OSC1)
- net PA10: now also SB15.1
- net PA13: now also SB14.1
- net PA14: now also SB6.1
- net PA9: now also SB11.1
- net PB3: now also SB9.2
- net STLINK_RX: now also JP4.1 (COMMON), SB11.2, U2.13 (PA3)
- net STLINK_TX: now also JP4.2 (NO), SB15.2, U2.12 (PA2)
- net STM_JTCK: now also SB5.2, U2.37 (JTCK/SWCLK)
- net STM_JTMS: now also SB13.2, U2.34 (JTMS/SWDIO)
- net STM_RST: now also C9.2, R21.1, SB10.2, U2.7 (NRST)
- net SWIM: now also U2.22 (PB11), U2.45 (PB8)
- net SWIM_IN: now also U2.21 (PB10), U2.43 (PB7), U2.46 (PB9)
- net SWIM_RST: now also U2.42 (PB6)
- net SWIM_RST_IN: now also U2.41 (PB5)
- net T_JTCK: now also R14.2, SB4.1, U2.15 (PA5), U2.26 (PB13)
- net T_JTDI: now also U2.17 (PA7)
- net T_JTDO: now also U2.16 (PA6)
- net T_JTMS: now also R15.2, R16.2, SB8.1, U2.27 (PB14)
- net T_NRST: now also R17.2, SB12.1, U2.18 (PB0)
- net T_SWDIO_IN: now also R16.1, U2.25 (PB12)
- net T_SWO: now also R20.2, SB9.1, U2.31 (PA10)
- net U5V: now also CN1.1 (VCC), D2.1 (A)
- net USB_DM: now also R12.2, U2.32 (PA11)
- net USB_DP: now also R11.2, U2.33 (PA12)
- net VDD: now also JP3.2 (NO)
- new net: CN1.2 (D-), R12.1
- new net: CN2.4, R15.1
- new net: R8.2, U2.44 (BOOT0)
- new net: C3.2, U1.4 (BYPASS)
- new net: LD1.4, R3.1
- new net: LD2.1, R4.1
- new net: CN4.1, SB3.1, SB4.2
- new net: CN4.2, SB5.1, SB6.2
- new net: CN4.3, SB7.1, SB8.2
- new net: CN4.4, SB13.1, SB14.2
- new net: CN1.3 (D+), R10.1, R11.1
- new net: R7.2, U2.2 (PC13)
- new net: R28.1, U2.29 (PA8)
- new net: CN2.1, D1.1 (A), R5.1
- new net: CN2.2, R14.1
- new net: CN2.5, R17.1
- new net: CN2.6, R20.1
- new net: C5.1, C6.2, D3.1 (A), U1.5 (Vout)
- new net: CN1.4 (ID), R9.1
- new net: LD1.3, R1.2
- new net: R6.2, U2.3 (PC14)
- new net: D1.2 (K), R13.1
- new net: LD1.2, R2.2

Commit message: esd protection for usb data lines
Parts:
- removed C1, C27, C4, C46, C47, C6, C9: 100nF, 0402C, symbol MCD_TOOLS:U_ST_LINK_1_Capacitor_ST_MCD_TOOLS.SchLib
- removed C16, C17, C18: 20pF, 0402C, symbol MCD_TOOLS:U_ST_LINK_1_Capacitor_ST_MCD_TOOLS.SchLib
- removed C2: 1µF_X5R_0603, 0603C, symbol MB963_1:U_ST_LINK_1_CAP SMD 0603 X5R 1µF 25V 10%_MB963_1.SCHLIB
- removed C3: 10nF_X7R_0603, 0603C, symbol MB963_1:U_ST_LINK_1_CAP SMD 0603 X7R 10000PF 50V 10%_MB963_1.SCHLIB
- removed C5: 1µF_X5R_0603, 0603C, symbol MB963_1:U_ST_LINK_3_CAP SMD 0603 X5R 1µF 25V 10%_MB963_1.SCHLIB
- removed CN1: USB-MINI-typeB, USB-MINI-B-SMD, symbol MCD_TOOLS:U_ST_LINK_0_USB-MINI-typeB connector_MCD_TOOLS.SchLib_0
- removed CN2: Header 6, HDR1X6, symbol Miscellaneous Connectors:U_ST_LINK_0_mirrored_Header 6_Miscellaneous Connectors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
- removed CN4: Header 4, Header 4, symbol MB963_1:U_ST_LINK_3_mirrored_Header 4_MB963_1.SCHLIB
- removed D1, D2, D3: BAT60JFILM, SOD323/A, symbol MCD_TOOLS:U_ST_LINK_0_BAT60JFILM_MCD_TOOLS.SchLib
- removed HW1, HW2, HW3, HW4, HW5: Shunt Black 2.54mm, symbol MB1075:U_ST_LINK_0_Shunt Black 2.54mm_MB1075.SCHLIB
- removed JP1, JP2, JP3: (no value), SIP2/2.54, symbol *:U_ST_LINK_0_JP2_*
- removed JP4: JP2, SIP2/2.54, symbol MCD_TOOLS:U_ST_LINK_1_JP2_MCD_TOOLS.SchLib
- removed LD1: LD_BICOLOR_CMS, HSMF-A201, symbol MCD_TOOLS:U_ST_LINK_0_mirrored_LD_BICOLOR_CMS_MCD_TOOLS.SchLib
- removed LD2: LED, red, 0603D, symbol MCD_TOOLS:U_ST_LINK_0_LED_red_MCD_TOOLS.SchLib_0
- removed R1, R2, R28: 100, 0402R, symbol MCD_TOOLS:U_ST_LINK_0_Resistor_ST_MCD_TOOLS.SchLib
- removed R10: 1K5, 0402R, symbol MCD_TOOLS:U_ST_LINK_0_Resistor_ST_MCD_TOOLS.SchLib
- removed R11, R12, R3: 0, 0402R, symbol MCD_TOOLS:U_ST_LINK_0_Resistor_ST_MCD_TOOLS.SchLib
- removed R13: [NA], 0402R, symbol MCD_TOOLS:U_ST_LINK_0_Resistor_ST_MCD_TOOLS.SchLib
- removed R14, R15, R17, R20: 22, 0402R, symbol MCD_TOOLS:U_ST_LINK_0_Resistor_ST_MCD_TOOLS.SchLib
- removed R16: 100, 0402R, symbol MCD_TOOLS:U_ST_LINK_1_Resistor_ST_MCD_TOOLS.SchLib
- removed R18, R19: 4K7, 0402R, symbol MCD_TOOLS:U_ST_LINK_0_Resistor_ST_MCD_TOOLS.SchLib
- removed R21: 100K, 0402R, symbol MCD_TOOLS:U_ST_LINK_1_Resistor_ST_MCD_TOOLS.SchLib
- removed R4: 1K, 0402R, symbol MCD_TOOLS:U_ST_LINK_1_Resistor_ST_MCD_TOOLS.SchLib
- removed R5: 10K, 0402R, symbol MCD_TOOLS:U_ST_LINK_1_Resistor_ST_MCD_TOOLS.SchLib
- removed R6, R7: 10K, 0402R, symbol MCD_TOOLS:U_ST_LINK_0_Resistor_ST_MCD_TOOLS.SchLib
- removed R8, R9: 100K, 0402R, symbol MCD_TOOLS:U_ST_LINK_0_Resistor_ST_MCD_TOOLS.SchLib
- removed SB10: Circuit Breaker, JP2_SMD, symbol MB915:U_ST_LINK_1_Circuit Breaker_MB915.SCHLIB
- removed SB11, SB15, SB9: Circuit Breaker, JP2_SMD, symbol MCD_TOOLS:U_ST_LINK_0_Circuit Breaker_MCD_TOOLS.SCHLIB
- removed SB12, SB13, SB14, SB3, SB4, SB5, SB6, SB7, SB8: Circuit Breaker, JP2_SMD, symbol MB915:U_ST_LINK_0_Circuit Breaker_MB915.SCHLIB
- removed U1: LD3985M33R, SOT-23-5L, symbol MCD_TOOLS:U_ST_LINK_0_LD3985M33R_MCD_TOOLS.SchLib
- removed U2: STM32F103CBT6, QFP48 7x7, symbol MCD_TOOLS:U_ST_LINK_0_STM32F103CBT6_MCD_TOOLS.SchLib
- removed X1: 8MHz, XTAL1, symbol MCD_TOOLS:U_ST_LINK_0_XTAL_MCD_TOOLS.SchLib_0
- added C (x7): 100nF, 0402C, symbol MCD_TOOLS:root_1_Capacitor_ST_MCD_TOOLS.SchLib
- added C (x3): 20pF, 0402C, symbol MCD_TOOLS:root_1_Capacitor_ST_MCD_TOOLS.SchLib
- added C: 10nF_X7R_0603, 0603C, symbol MB963_1:root_1_CAP SMD 0603 X7R 10000PF 50V 10%_MB963_1.SCHLIB
- added C: 1µF_X5R_0603, 0603C, symbol MB963_1:root_1_CAP SMD 0603 X5R 1µF 25V 10%_MB963_1.SCHLIB
- added C: 1µF_X5R_0603, 0603C, symbol MB963_1:root_3_CAP SMD 0603 X5R 1µF 25V 10%_MB963_1.SCHLIB
- added CN: Header 6, HDR1X6, symbol Miscellaneous Connectors:root_0_mirrored_Header 6_Miscellaneous Connectors.IntL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
- added CN: Header 4, Header 4, symbol MB963_1:root_3_mirrored_Header 4_MB963_1.SCHLIB
- added CN: USB-MINI-typeB, USB-MINI-B-SMD, symbol MCD_TOOLS:root_0_USB-MINI-typeB connector_MCD_TOOLS.SchLib_0
- added D (x3): BAT60JFILM, SOD323/A, symbol MCD_TOOLS:root_0_BAT60JFILM_MCD_TOOLS.SchLib
- added HW (x5): Shunt Black 2.54mm, symbol MB1075:root_0_Shunt Black 2.54mm_MB1075.SCHLIB
- added JP (x3): (no value), SIP2/2.54, symbol *:root_0_JP2_*
- added JP: JP2, SIP2/2.54, symbol MCD_TOOLS:root_1_JP2_MCD_TOOLS.SchLib
- added LD: LED, red, 0603D, symbol MCD_TOOLS:root_0_LED_red_MCD_TOOLS.SchLib_0
- added LD: LD_BICOLOR_CMS, HSMF-A201, symbol MCD_TOOLS:root_0_mirrored_LD_BICOLOR_CMS_MCD_TOOLS.SchLib
- added R: 1K5, 0402R, symbol MCD_TOOLS:root_0_Resistor_ST_MCD_TOOLS.SchLib
- added R (x2): 10K, 0402R, symbol MCD_TOOLS:root_0_Resistor_ST_MCD_TOOLS.SchLib
- added R: 100K, 0402R, symbol MCD_TOOLS:root_1_Resistor_ST_MCD_TOOLS.SchLib
- added R (x2): 4K7, 0402R, symbol MCD_TOOLS:root_0_Resistor_ST_MCD_TOOLS.SchLib
- added R: 100, 0402R, symbol MCD_TOOLS:root_1_Resistor_ST_MCD_TOOLS.SchLib
- added R (x3): 100, 0402R, symbol MCD_TOOLS:root_0_Resistor_ST_MCD_TOOLS.SchLib
- added R: 1K, 0402R, symbol MCD_TOOLS:root_1_Resistor_ST_MCD_TOOLS.SchLib
- added R: [NA], 0402R, symbol MCD_TOOLS:root_0_Resistor_ST_MCD_TOOLS.SchLib
- added R (x2): 100K, 0402R, symbol MCD_TOOLS:root_0_Resistor_ST_MCD_TOOLS.SchLib
- added R (x4): 22, 0402R, symbol MCD_TOOLS:root_0_Resistor_ST_MCD_TOOLS.SchLib
- added R: 10K, 0402R, symbol MCD_TOOLS:root_1_Resistor_ST_MCD_TOOLS.SchLib
- added R (x3): 0, 0402R, symbol MCD_TOOLS:root_0_Resistor_ST_MCD_TOOLS.SchLib
- added SB (x9): Circuit Breaker, JP2_SMD, symbol MB915:root_0_Circuit Breaker_MB915.SCHLIB
- added SB (x3): Circuit Breaker, JP2_SMD, symbol MCD_TOOLS:root_0_Circuit Breaker_MCD_TOOLS.SCHLIB
- added SB: Circuit Breaker, JP2_SMD, symbol MB915:root_1_Circuit Breaker_MB915.SCHLIB
- added U: STM32F103CBT6, QFP48 7x7, symbol MCD_TOOLS:root_0_STM32F103CBT6_MCD_TOOLS.SchLib
- added U: LD3985M33R, SOT-23-5L, symbol MCD_TOOLS:root_0_LD3985M33R_MCD_TOOLS.SchLib
- added X: 8MHz, XTAL1, symbol MCD_TOOLS:root_0_XTAL_MCD_TOOLS.SchLib_0
Connections:
- net 3V: now also C.2, C.2, C.2, C.2, D.2 (K), JP.1 (COMMON), R.1, R.2, R.2, R.2, R.2, SB.2, U.1 (VBAT), U.24 (VDD_1), U.36 (VDD_2), U.48 (VDD_3), U.9 (VDDA)
- net 5V: now also C.2, C.2, D.2 (K), U.1 (Vin), U.3 (CE)
- net AIN_1: now also R.2, R.2, R.2, U.10 (PA0)
- net GND: now also C.1, C.1, C.1, C.1, C.1, C.1, C.1, C.1, C.1, C.1, C.2, C.2, C.2, CN.3, CN.5 (GND), CN.6 (SHELL), JP.1 (COMMON), JP.1 (COMMON), JP.2 (NO), JP.2 (NO), LD.1, LD.2, R.1, R.1, R.1, R.1, R.2, R.2, SB.1, SB.2, U.2 (GND), U.20 (PB2/BOOT1), U.23 (VSS_1), U.35 (VSS_2), U.47 (VSS_3), U.8 (VSSA)
- net LED_STLINK: now also R.1, R.1, U.30 (PA9)
- net MCO: now also C.2, R.2
- net NRST: now also SB.2
- net OSC_IN: now also C.1, U.5 (OSCIN), X.2 (OSC2)
- net OSC_OUT: now also C.1, U.6 (OSCOUT), X.1 (OSC1)
- net PA10: now also SB.1
- net PA13: now also SB.1
- net PA14: now also SB.1
- net PA9: now also SB.1
- net PB3: now also SB.2
- net STLINK_RX: now also JP.1 (COMMON), SB.2, U.13 (PA3)
- net STLINK_TX: now also JP.2 (NO), SB.2, U.12 (PA2)
- net STM_JTCK: now also SB.2, U.37 (JTCK/SWCLK)
- net STM_JTMS: now also SB.2, U.34 (JTMS/SWDIO)
- net STM_RST: now also C.2, R.1, SB.2, U.7 (NRST)
- net SWIM: now also U.22 (PB11), U.45 (PB8)
- net SWIM_IN: now also U.21 (PB10), U.43 (PB7), U.46 (PB9)
- net SWIM_RST: now also U.42 (PB6)
- net SWIM_RST_IN: now also U.41 (PB5)
- net T_JTCK: now also R.2, SB.1, U.15 (PA5), U.26 (PB13)
- net T_JTDI: now also U.17 (PA7)
- net T_JTDO: now also U.16 (PA6)
- net T_JTMS: now also R.2, R.2, SB.1, U.27 (PB14)
- net T_NRST: now also R.2, SB.1, U.18 (PB0)
- net T_SWDIO_IN: now also R.1, U.25 (PB12)
- net T_SWO: now also R.2, SB.1, U.31 (PA10)
- net U5V: now also CN.1 (VCC), D.1 (A)
- net USB_DM: now also R.2, U.32 (PA11)
- net USB_DP: now also R.2, U.33 (PA12)
- net VDD: now also JP.2 (NO)
- new net: CN.1, SB.1, SB.2
- new net: CN.3 (D+), R.1, R.1
- new net: R.2, U.2 (PC13)
- new net: CN.1, D.1 (A), R.1
- new net: D.2 (K), R.1
- new net: R.1, U.29 (PA8)
- new net: LD.1, R.1
- new net: R.2, U.3 (PC14)
- new net: CN.4, SB.1, SB.2
- new net: R.2, U.44 (BOOT0)
- new net: C.2, U.4 (BYPASS)
- new net: CN.4 (ID), R.1
- new net: CN.4, R.1
- new net: CN.2, R.1
- new net: CN.5, R.1
- new net: CN.6, R.1
- new net: LD.3, R.2
- new net: CN.3, SB.1, SB.2
- new net: CN.2, SB.1, SB.2
- new net: C.1, C.2, D.1 (A), U.5 (Vout)
- new net: CN.2 (D-), R.1
- new net: LD.4, R.1
- new net: LD.2, R.2

Commit message: measuring trace lengths, looks ok so far! almost done
Parts:
- removed C (x7): 100nF, 0402C, symbol MCD_TOOLS:root_1_Capacitor_ST_MCD_TOOLS.SchLib
- removed C (x3): 20pF, 0402C, symbol MCD_TOOLS:root_1_Capacitor_ST_MCD_TOOLS.SchLib
- removed D (x3): BAT60JFILM, SOD323/A, symbol MCD_TOOLS:root_0_BAT60JFILM_MCD_TOOLS.SchLib
- removed HW (x5): Shunt Black 2.54mm, symbol MB1075:root_0_Shunt Black 2.54mm_MB1075.SCHLIB
- removed JP (x3): (no value), SIP2/2.54, symbol *:root_0_JP2_*
- removed R: 1K5, 0402R, symbol MCD_TOOLS:root_0_Resistor_ST_MCD_TOOLS.SchLib
- removed R (x2): 10K, 0402R, symbol MCD_TOOLS:root_0_Resistor_ST_MCD_TOOLS.SchLib
- removed R: 100K, 0402R, symbol MCD_TOOLS:root_1_Resistor_ST_MCD_TOOLS.SchLib
- removed R (x2): 4K7, 0402R, symbol MCD_TOOLS:root_0_Resistor_ST_MCD_TOOLS.SchLib
- removed R: 100, 0402R, symbol MCD_TOOLS:root_1_Resistor_ST_MCD_TOOLS.SchLib
- removed R (x3): 100, 0402R, symbol MCD_TOOLS:root_0_Resistor_ST_MCD_TOOLS.SchLib
- removed R: 1K, 0402R, symbol MCD_TOOLS:root_1_Resistor_ST_MCD_TOOLS.SchLib
- removed R: [NA], 0402R, symbol MCD_TOOLS:root_0_Resistor_ST_MCD_TOOLS.SchLib
- removed R (x2): 100K, 0402R, symbol MCD_TOOLS:root_0_Resistor_ST_MCD_TOOLS.SchLib
- removed R (x4): 22, 0402R, symbol MCD_TOOLS:root_0_Resistor_ST_MCD_TOOLS.SchLib
- removed R: 10K, 0402R, symbol MCD_TOOLS:root_1_Resistor_ST_MCD_TOOLS.SchLib
- removed R (x3): 0, 0402R, symbol MCD_TOOLS:root_0_Resistor_ST_MCD_TOOLS.SchLib
- removed SB (x9): Circuit Breaker, JP2_SMD, symbol MB915:root_0_Circuit Breaker_MB915.SCHLIB
- removed SB (x3): Circuit Breaker, JP2_SMD, symbol MCD_TOOLS:root_0_Circuit Breaker_MCD_TOOLS.SCHLIB
- added C (x7): 100nF, 0402C, symbol MCD_TOOLS:root_1_Capacitor_ST_MCD_TOOLS.SchLib
- added C (x3): 20pF, 0402C, symbol MCD_TOOLS:root_1_Capacitor_ST_MCD_TOOLS.SchLib
- added D (x3): BAT60JFILM, SOD323/A, symbol MCD_TOOLS:root_0_BAT60JFILM_MCD_TOOLS.SchLib
- added HW (x5): Shunt Black 2.54mm, symbol MB1075:root_0_Shunt Black 2.54mm_MB1075.SCHLIB
- added JP (x3): (no value), SIP2/2.54, symbol *:root_0_JP2_*
- added R (x4): 22, 0402R, symbol MCD_TOOLS:root_0_Resistor_ST_MCD_TOOLS.SchLib
- added R: 10K, 0402R, symbol MCD_TOOLS:root_1_Resistor_ST_MCD_TOOLS.SchLib
- added R (x3): 100, 0402R, symbol MCD_TOOLS:root_0_Resistor_ST_MCD_TOOLS.SchLib
- added R: 1K5, 0402R, symbol MCD_TOOLS:root_0_Resistor_ST_MCD_TOOLS.SchLib
- added R: 1K, 0402R, symbol MCD_TOOLS:root_1_Resistor_ST_MCD_TOOLS.SchLib
- added R (x2): 4K7, 0402R, symbol MCD_TOOLS:root_0_Resistor_ST_MCD_TOOLS.SchLib
- added R: [NA], 0402R, symbol MCD_TOOLS:root_0_Resistor_ST_MCD_TOOLS.SchLib
- added R (x3): 0, 0402R, symbol MCD_TOOLS:root_0_Resistor_ST_MCD_TOOLS.SchLib
- added R (x2): 100K, 0402R, symbol MCD_TOOLS:root_0_Resistor_ST_MCD_TOOLS.SchLib
- added R (x2): 10K, 0402R, symbol MCD_TOOLS:root_0_Resistor_ST_MCD_TOOLS.SchLib
- added R: 100, 0402R, symbol MCD_TOOLS:root_1_Resistor_ST_MCD_TOOLS.SchLib
- added R: 100K, 0402R, symbol MCD_TOOLS:root_1_Resistor_ST_MCD_TOOLS.SchLib
- added SB (x9): Circuit Breaker, JP2_SMD, symbol MB915:root_0_Circuit Breaker_MB915.SCHLIB
- added SB (x3): Circuit Breaker, JP2_SMD, symbol MCD_TOOLS:root_0_Circuit Breaker_MCD_TOOLS.SCHLIB
Connections:
- net 3V: now also C.2, C.2, C.2, C.2, D.2 (K), JP.1 (COMMON), R.1, R.2, R.2, R.2, R.2, SB.2
- net 5V: now also C.2, D.2 (K)
- net AIN_1: now also R.2, R.2, R.2
- net GND: now also C.1, C.1, C.1, C.1, C.1, C.1, C.1, C.1, C.2, C.2, JP.1 (COMMON), JP.1 (COMMON), JP.2 (NO), JP.2 (NO), R.1, R.1, R.1, R.1, R.2, R.2, SB.2
- net LED_STLINK: now also R.1, R.1
- net MCO: now also C.2, R.2
- net NRST: now also SB.2
- net OSC_IN: now also C.1
- net OSC_OUT: now also C.1
- net PA10: now also SB.1
- net PA13: now also SB.1
- net PA14: now also SB.1
- net PA9: now also SB.1
- net PB3: now also SB.2
- net STLINK_RX: now also SB.2
- net STLINK_TX: now also SB.2
- net STM_JTCK: now also SB.2
- net STM_JTMS: now also SB.2
- net STM_RST: now also C.2, R.1
- net T_JTCK: now also R.2, SB.1
- net T_JTMS: now also R.2, R.2, SB.1
- net T_NRST: now also R.2, SB.1
- net T_SWDIO_IN: now also R.1
- net T_SWO: now also R.2, SB.1
- net U5V: now also D.1 (A)
- net USB_DM: now also R.2
- net USB_DP: now also R.2
- net VDD: now also JP.2 (NO)
- net at CN.1: now also SB.1, SB.2
- net at CN.3 (D+): now also R.1, R.1
- net at U.2 (PC13): now also R.2
- net at CN.1: now also D.1 (A), R.1
- net at U.29 (PA8): now also R.1
- net at LD.1: now also R.1
- net at U.3 (PC14): now also R.2
- net at CN.4: now also SB.1, SB.2
- net at U.44 (BOOT0): now also R.2
- net at CN.4 (ID): now also R.1
- net at CN.4: now also R.1
- net at CN.2: now also R.1
- net at CN.5: now also R.1
- net at CN.6: now also R.1
- net at LD.3: now also R.2
- net at CN.3: now also SB.1, SB.2
- net at CN.2: now also SB.1, SB.2
- net at C.1, U.5 (Vout): now also C.2, D.1 (A)
- net at CN.2 (D-): now also R.1
- net at LD.4: now also R.1
- net at LD.2: now also R.2
- new net: D.2 (K), R.1
