File: docs/mb1075_bdp/MB1075E/Altium_Designer/USB_OTG_FS.kicad_sch (KiCad schematic)
At the start: 18 parts, among them CN6 USB-MICRO-AB, T1 9013-SOT23, U7 EMIF02-USB03F2, U8 STMPS2141STR

Commit message: save before i break everything out instead idk why i didnt do that
Parts:
- removed C53: 4.7uF, TAN-A, symbol Miscellaneous Devices:U_USB_OTG_FS_3_Cap Pol1_Miscellaneous Devices.IntLib
- removed CN6: USB-MICRO-AB, CON_USBMICROAB_MOLEX_47590-0001_H3, symbol MCD_TOOLS:U_USB_OTG_FS_0_USB-MICRO-AB_MCD_TOOLS.SchLib
- removed LD5: Green, 0603D, symbol Miscellaneous Devices:U_USB_OTG_FS_3_LED2_Miscellaneous Devices.IntLib
- removed LD6: Red, 0603D, symbol Miscellaneous Devices:U_USB_OTG_FS_3_LED2_Miscellaneous Devices.IntLib
- removed R63, R64: 22, 0402R, symbol MCD_TOOLS:U_USB_OTG_FS_0_Resistor_ST_MCD_TOOLS.SchLib
- removed R65, R68: 47K, 0402R, symbol MCD_TOOLS:U_USB_OTG_FS_1_Resistor_ST_MCD_TOOLS.SchLib
- removed R66: [N/A], 0402R, symbol MCD_TOOLS:U_USB_OTG_FS_0_Resistor_ST_MCD_TOOLS.SchLib
- removed R67, R69, R72: 0, 0402R, symbol MCD_TOOLS:U_USB_OTG_FS_0_Resistor_ST_MCD_TOOLS.SchLib
- removed R70: 330, 0603R, symbol MCD_TOOLS:U_USB_OTG_FS_1_Resistor_ST_MCD_TOOLS.SchLib
- removed R71: 10K, 0402R, symbol MCD_TOOLS:U_USB_OTG_FS_1_Resistor_ST_MCD_TOOLS.SchLib
- removed R73: 620, 0603R, symbol MCD_TOOLS:U_USB_OTG_FS_1_Resistor_ST_MCD_TOOLS.SchLib
- removed T1: 9013-SOT23, SOT-23, symbol MCD_TOOLS:U_USB_OTG_FS_0_9013-SOT23_MCD_TOOLS.SchLib
- removed U7: EMIF02-USB03F2, Flip Chip, symbol MCD_TOOLS:U_USB_OTG_FS_0_EMIF02-USB03F2_MCD_TOOLS.SchLib
- removed U8: STMPS2141STR, SOT23-5L, symbol MCD_TOOLS:U_USB_OTG_FS_0_STMPS2141STR_MCD_TOOLS.SchLib
- added C53: 4.7uF, TAN-A, symbol Miscellaneous Devices:root_3_Cap Pol1_Miscellaneous Devices.IntLib
- added CN6: USB-MICRO-AB, CON_USBMICROAB_MOLEX_47590-0001_H3, symbol MCD_TOOLS:root_0_USB-MICRO-AB_MCD_TOOLS.SchLib
- added LD5: Green, 0603D, symbol Miscellaneous Devices:root_3_LED2_Miscellaneous Devices.IntLib
- added LD6: Red, 0603D, symbol Miscellaneous Devices:root_3_LED2_Miscellaneous Devices.IntLib
- added R63, R64: 22, 0402R, symbol MCD_TOOLS:root_0_Resistor_ST_MCD_TOOLS.SchLib
- added R65, R68: 47K, 0402R, symbol MCD_TOOLS:root_1_Resistor_ST_MCD_TOOLS.SchLib
- added R66: [N/A], 0402R, symbol MCD_TOOLS:root_0_Resistor_ST_MCD_TOOLS.SchLib
- added R67, R69, R72: 0, 0402R, symbol MCD_TOOLS:root_0_Resistor_ST_MCD_TOOLS.SchLib
- added R70: 330, 0603R, symbol MCD_TOOLS:root_1_Resistor_ST_MCD_TOOLS.SchLib
- added R71: 10K, 0402R, symbol MCD_TOOLS:root_1_Resistor_ST_MCD_TOOLS.SchLib
- added R73: 620, 0603R, symbol MCD_TOOLS:root_1_Resistor_ST_MCD_TOOLS.SchLib
- added T1: 9013-SOT23, SOT-23, symbol MCD_TOOLS:root_0_9013-SOT23_MCD_TOOLS.SchLib
- added U7: EMIF02-USB03F2, Flip Chip, symbol MCD_TOOLS:root_0_EMIF02-USB03F2_MCD_TOOLS.SchLib
- added U8: STMPS2141STR, SOT23-5L, symbol MCD_TOOLS:root_0_STMPS2141STR_MCD_TOOLS.SchLib
Connections:
- net 3V: now also R68.2, R70.2, R71.2, R73.2
- net 5V: now also U8.5 (IN)
- net GND: now also C53.2, CN6.5 (GND), CN6.6 (Shield), R66.2, T1.2 (E), U7.D2 (GND), U8.2 (GND)
- net OTG_FS_DM: now also R64.1, U7.D3 (D-out)
- net OTG_FS_DP: now also R63.1, U7.C3 (D+out)
- net OTG_FS_ID: now also R67.1
- net OTG_FS_OC: now also R69.2
- net OTG_FS_PSO: now also R72.1
- net VBUS_FS: now also C53.1, CN6.1 (VBUS), R65.2, U7.B3 (Vbus), U8.1 (OUT)
- new net: CN6.3 (DP), R63.2, U7.C1 (D+in)
- new net: R65.1, R66.1, T1.1 (B)
- new net: LD5.2 (K), T1.3 (C)
- new net: LD6.2 (K), R68.1, R69.1, U8.3 (~{FAULT})
- new net: R71.1, R72.2, U8.4 (~{EN})
- new net: LD6.1 (A), R73.1
- new net: CN6.4 (ID), R67.2, U7.A3 (ID)
- new net: CN6.2 (DM), R64.2, U7.D1 (D-in)
- new net: LD5.1 (A), R70.1

Commit message: KILL ME!!!!!!!!!!!
Parts:
- removed C53: 4.7uF, TAN-A, symbol Miscellaneous Devices:root_3_Cap Pol1_Miscellaneous Devices.IntLib
- removed CN6: USB-MICRO-AB, CON_USBMICROAB_MOLEX_47590-0001_H3, symbol MCD_TOOLS:root_0_USB-MICRO-AB_MCD_TOOLS.SchLib
- removed LD5: Green, 0603D, symbol Miscellaneous Devices:root_3_LED2_Miscellaneous Devices.IntLib
- removed LD6: Red, 0603D, symbol Miscellaneous Devices:root_3_LED2_Miscellaneous Devices.IntLib
- removed R63, R64: 22, 0402R, symbol MCD_TOOLS:root_0_Resistor_ST_MCD_TOOLS.SchLib
- removed R65, R68: 47K, 0402R, symbol MCD_TOOLS:root_1_Resistor_ST_MCD_TOOLS.SchLib
- removed R66: [N/A], 0402R, symbol MCD_TOOLS:root_0_Resistor_ST_MCD_TOOLS.SchLib
- removed R67, R69, R72: 0, 0402R, symbol MCD_TOOLS:root_0_Resistor_ST_MCD_TOOLS.SchLib
- removed R70: 330, 0603R, symbol MCD_TOOLS:root_1_Resistor_ST_MCD_TOOLS.SchLib
- removed R71: 10K, 0402R, symbol MCD_TOOLS:root_1_Resistor_ST_MCD_TOOLS.SchLib
- removed R73: 620, 0603R, symbol MCD_TOOLS:root_1_Resistor_ST_MCD_TOOLS.SchLib
- removed T1: 9013-SOT23, SOT-23, symbol MCD_TOOLS:root_0_9013-SOT23_MCD_TOOLS.SchLib
- removed U7: EMIF02-USB03F2, Flip Chip, symbol MCD_TOOLS:root_0_EMIF02-USB03F2_MCD_TOOLS.SchLib
- removed U8: STMPS2141STR, SOT23-5L, symbol MCD_TOOLS:root_0_STMPS2141STR_MCD_TOOLS.SchLib
- added C53: 4.7uF, TAN-A, symbol Miscellaneous Devices:U_USB_OTG_FS_3_Cap Pol1_Miscellaneous Devices.IntLib
- added CN6: USB-MICRO-AB, CON_USBMICROAB_MOLEX_47590-0001_H3, symbol MCD_TOOLS:U_USB_OTG_FS_0_USB-MICRO-AB_MCD_TOOLS.SchLib
- added LD5: Green, 0603D, symbol Miscellaneous Devices:U_USB_OTG_FS_3_LED2_Miscellaneous Devices.IntLib
- added LD6: Red, 0603D, symbol Miscellaneous Devices:U_USB_OTG_FS_3_LED2_Miscellaneous Devices.IntLib
- added R63, R64: 22, 0402R, symbol MCD_TOOLS:U_USB_OTG_FS_0_Resistor_ST_MCD_TOOLS.SchLib
- added R65, R68: 47K, 0402R, symbol MCD_TOOLS:U_USB_OTG_FS_1_Resistor_ST_MCD_TOOLS.SchLib
- added R66: [N/A], 0402R, symbol MCD_TOOLS:U_USB_OTG_FS_0_Resistor_ST_MCD_TOOLS.SchLib
- added R67, R69, R72: 0, 0402R, symbol MCD_TOOLS:U_USB_OTG_FS_0_Resistor_ST_MCD_TOOLS.SchLib
- added R70: 330, 0603R, symbol MCD_TOOLS:U_USB_OTG_FS_1_Resistor_ST_MCD_TOOLS.SchLib
- added R71: 10K, 0402R, symbol MCD_TOOLS:U_USB_OTG_FS_1_Resistor_ST_MCD_TOOLS.SchLib
- added R73: 620, 0603R, symbol MCD_TOOLS:U_USB_OTG_FS_1_Resistor_ST_MCD_TOOLS.SchLib
- added T1: 9013-SOT23, SOT-23, symbol MCD_TOOLS:U_USB_OTG_FS_0_9013-SOT23_MCD_TOOLS.SchLib
- added U7: EMIF02-USB03F2, Flip Chip, symbol MCD_TOOLS:U_USB_OTG_FS_0_EMIF02-USB03F2_MCD_TOOLS.SchLib
- added U8: STMPS2141STR, SOT23-5L, symbol MCD_TOOLS:U_USB_OTG_FS_0_STMPS2141STR_MCD_TOOLS.SchLib
Connections:
- net 3V: now also R68.2, R70.2, R71.2, R73.2
- net 5V: now also U8.5 (IN)
- net GND: now also C53.2, CN6.5 (GND), CN6.6 (Shield), R66.2, T1.2 (E), U7.D2 (GND), U8.2 (GND)
- net OTG_FS_DM: now also R64.1, U7.D3 (D-out)
- net OTG_FS_DP: now also R63.1, U7.C3 (D+out)
- net OTG_FS_ID: now also R67.1
- net OTG_FS_OC: now also R69.2
- net OTG_FS_PSO: now also R72.1
- net VBUS_FS: now also C53.1, CN6.1 (VBUS), R65.2, U7.B3 (Vbus), U8.1 (OUT)
- new net: LD6.2 (K), R68.1, R69.1, U8.3 (~{FAULT})
- new net: CN6.4 (ID), R67.2, U7.A3 (ID)
- new net: CN6.3 (DP), R63.2, U7.C1 (D+in)
- new net: CN6.2 (DM), R64.2, U7.D1 (D-in)
- new net: LD6.1 (A), R73.1
- new net: R65.1, R66.1, T1.1 (B)
- new net: LD5.2 (K), T1.3 (C)
- new net: R71.1, R72.2, U8.4 (~{EN})
- new net: LD5.1 (A), R70.1

Commit message: esd protection for usb data lines
Parts:
- removed C53: 4.7uF, TAN-A, symbol Miscellaneous Devices:U_USB_OTG_FS_3_Cap Pol1_Miscellaneous Devices.IntLib
- removed CN6: USB-MICRO-AB, CON_USBMICROAB_MOLEX_47590-0001_H3, symbol MCD_TOOLS:U_USB_OTG_FS_0_USB-MICRO-AB_MCD_TOOLS.SchLib
- removed LD5: Green, 0603D, symbol Miscellaneous Devices:U_USB_OTG_FS_3_LED2_Miscellaneous Devices.IntLib
- removed LD6: Red, 0603D, symbol Miscellaneous Devices:U_USB_OTG_FS_3_LED2_Miscellaneous Devices.IntLib
- removed R63, R64: 22, 0402R, symbol MCD_TOOLS:U_USB_OTG_FS_0_Resistor_ST_MCD_TOOLS.SchLib
- removed R65, R68: 47K, 0402R, symbol MCD_TOOLS:U_USB_OTG_FS_1_Resistor_ST_MCD_TOOLS.SchLib
- removed R66: [N/A], 0402R, symbol MCD_TOOLS:U_USB_OTG_FS_0_Resistor_ST_MCD_TOOLS.SchLib
- removed R67, R69, R72: 0, 0402R, symbol MCD_TOOLS:U_USB_OTG_FS_0_Resistor_ST_MCD_TOOLS.SchLib
- removed R70: 330, 0603R, symbol MCD_TOOLS:U_USB_OTG_FS_1_Resistor_ST_MCD_TOOLS.SchLib
- removed R71: 10K, 0402R, symbol MCD_TOOLS:U_USB_OTG_FS_1_Resistor_ST_MCD_TOOLS.SchLib
- removed R73: 620, 0603R, symbol MCD_TOOLS:U_USB_OTG_FS_1_Resistor_ST_MCD_TOOLS.SchLib
- removed T1: 9013-SOT23, SOT-23, symbol MCD_TOOLS:U_USB_OTG_FS_0_9013-SOT23_MCD_TOOLS.SchLib
- removed U7: EMIF02-USB03F2, Flip Chip, symbol MCD_TOOLS:U_USB_OTG_FS_0_EMIF02-USB03F2_MCD_TOOLS.SchLib
- removed U8: STMPS2141STR, SOT23-5L, symbol MCD_TOOLS:U_USB_OTG_FS_0_STMPS2141STR_MCD_TOOLS.SchLib
- added C53: 4.7uF, TAN-A, symbol Miscellaneous Devices:root_3_Cap Pol1_Miscellaneous Devices.IntLib
- added CN6: USB-MICRO-AB, CON_USBMICROAB_MOLEX_47590-0001_H3, symbol MCD_TOOLS:root_0_USB-MICRO-AB_MCD_TOOLS.SchLib
- added LD5: Green, 0603D, symbol Miscellaneous Devices:root_3_LED2_Miscellaneous Devices.IntLib
- added LD6: Red, 0603D, symbol Miscellaneous Devices:root_3_LED2_Miscellaneous Devices.IntLib
- added R63, R64: 22, 0402R, symbol MCD_TOOLS:root_0_Resistor_ST_MCD_TOOLS.SchLib
- added R65, R68: 47K, 0402R, symbol MCD_TOOLS:root_1_Resistor_ST_MCD_TOOLS.SchLib
- added R66: [N/A], 0402R, symbol MCD_TOOLS:root_0_Resistor_ST_MCD_TOOLS.SchLib
- added R67, R69, R72: 0, 0402R, symbol MCD_TOOLS:root_0_Resistor_ST_MCD_TOOLS.SchLib
- added R70: 330, 0603R, symbol MCD_TOOLS:root_1_Resistor_ST_MCD_TOOLS.SchLib
- added R71: 10K, 0402R, symbol MCD_TOOLS:root_1_Resistor_ST_MCD_TOOLS.SchLib
- added R73: 620, 0603R, symbol MCD_TOOLS:root_1_Resistor_ST_MCD_TOOLS.SchLib
- added T1: 9013-SOT23, SOT-23, symbol MCD_TOOLS:root_0_9013-SOT23_MCD_TOOLS.SchLib
- added U7: EMIF02-USB03F2, Flip Chip, symbol MCD_TOOLS:root_0_EMIF02-USB03F2_MCD_TOOLS.SchLib
- added U8: STMPS2141STR, SOT23-5L, symbol MCD_TOOLS:root_0_STMPS2141STR_MCD_TOOLS.SchLib
Connections:
- net 3V: now also R68.2, R70.2, R71.2, R73.2
- net 5V: now also U8.5 (IN)
- net GND: now also C53.2, CN6.5 (GND), CN6.6 (Shield), R66.2, T1.2 (E), U7.D2 (GND), U8.2 (GND)
- net OTG_FS_DM: now also R64.1, U7.D3 (D-out)
- net OTG_FS_DP: now also R63.1, U7.C3 (D+out)
- net OTG_FS_ID: now also R67.1
- net OTG_FS_OC: now also R69.2
- net OTG_FS_PSO: now also R72.1
- net VBUS_FS: now also C53.1, CN6.1 (VBUS), R65.2, U7.B3 (Vbus), U8.1 (OUT)
- new net: R71.1, R72.2, U8.4 (~{EN})
- new net: R65.1, R66.1, T1.1 (B)
- new net: CN6.2 (DM), R64.2, U7.D1 (D-in)
- new net: CN6.4 (ID), R67.2, U7.A3 (ID)
- new net: CN6.3 (DP), R63.2, U7.C1 (D+in)
- new net: LD5.1 (A), R70.1
- new net: LD5.2 (K), T1.3 (C)
- new net: LD6.1 (A), R73.1
- new net: LD6.2 (K), R68.1, R69.1, U8.3 (~{FAULT})
